Commit message: Createt the Base for the Hardware Interface

File: description/ros2_control/melfa.ros2_control.xacro (robot description, xacro)
@@ -15,5 +15,5 @@
           </xacro:if>
           <xacro:unless value="${use_fake_hardware}">
-            <plugin>melfa_robot/MelfaHW</plugin>
+            <plugin>melfa_assita_ros2_hw/MelfaHW</plugin>
             <param name="robot_ip">${robot_ip}</param>
           </xacro:unless>

File: description/urdf/RV-5AS.urdf.xacro (robot description, xacro)
@@ -5,7 +5,7 @@
 <xacro:arg name="use_fake_hardware" default="true" />
 <xacro:arg name="robot_ip" default="127.0.0.1" />
-<xacro:include filename="$(find melfa_robot)/urdf/materials.xacro" />
-<xacro:include filename="$(find melfa_robot)/urdf/RV-5AS.gazebo" />
-<xacro:include filename="$(find melfa_robot)/ros2_control/melfa.ros2_control.xacro" />
+<xacro:include filename="$(find melfa_assita_ros2_hw)/urdf/materials.xacro" />
+<xacro:include filename="$(find melfa_assita_ros2_hw)/urdf/RV-5AS.gazebo" />
+<xacro:include filename="$(find melfa_assita_ros2_hw)/ros2_control/melfa.ros2_control.xacro" />
 <!-- Enable Gazebo Plugins -->
   <gazebo>
@@ -13,5 +13,5 @@
       <!-- <robot_param>robot_description</robot_param>
       <robot_param_node>robot_state_publisher</robot_param_node> -->
-      <parameters>$(find melfa_robot)/config/melfa_controller.yaml</parameters>
+      <parameters>$(find melfa_assita_ros2_hw)/config/melfa_controller.yaml</parameters>
     </plugin>
   </gazebo>
@@ -28,5 +28,5 @@
     <origin xyz="0 0 0" rpy="0 0 0"/>
     <geometry>
-      <mesh filename="package://melfa_robot/meshes/base_link.stl" scale="0.001 0.001 0.001"/>
+      <mesh filename="package://melfa_assita_ros2_hw/meshes/base_link.stl" scale="0.001 0.001 0.001"/>
       <cylinder radius="0.5" length="1.0"/>
     </geometry>
@@ -36,5 +36,5 @@
     <origin xyz="0 0 0" rpy="0 0 0"/>
     <geometry>
-      <mesh filename="package://melfa_robot/meshes/base_link.stl" scale="0.001 0.001 0.001"/>
+      <mesh filename="package://melfa_assita_ros2_hw/meshes/base_link.stl" scale="0.001 0.001 0.001"/>
     </geometry>
   </collision>
@@ -49,5 +49,5 @@
     <origin xyz="-0.000321 -0.000483 -0.169215" rpy="0 0 0"/>
     <geometry>
-      <mesh filename="package://melfa_robot/meshes/Link_1_1.stl" scale="0.001 0.001 0.001"/>
+      <mesh filename="package://melfa_assita_ros2_hw/meshes/Link_1_1.stl" scale="0.001 0.001 0.001"/>
     </geometry>
     <material name="silver"/>
@@ -56,5 +56,5 @@
     <origin xyz="-0.000321 -0.000483 -0.169215" rpy="0 0 0"/>
     <geometry>
-      <mesh filename="package://melfa_robot/meshes/Link_1_1.stl" scale="0.001 0.001 0.001"/>
+      <mesh filename="package://melfa_assita_ros2_hw/meshes/Link_1_1.stl" scale="0.001 0.001 0.001"/>
     </geometry>
   </collision>
@@ -69,5 +69,5 @@
     <origin xyz="-0.000321 -0.091983 -0.252215" rpy="0 0 0"/>
     <geometry>
-      <mesh filename="package://melfa_robot/meshes/Link_2_1.stl" scale="0.001 0.001 0.001"/>
+      <mesh filename="package://melfa_assita_ros2_hw/meshes/Link_2_1.stl" scale="0.001 0.001 0.001"/>
     </geometry>
     <material name="silver"/>
@@ -76,5 +76,5 @@
     <origin xyz="-0.000321 -0.091983 -0.252215" rpy="0 0 0"/>
     <geometry>
-      <mesh filename="package://melfa_robot/meshes/Link_2_1.stl" scale="0.001 0.001 0.001"/>
+      <mesh filename="package://melfa_assita_ros2_hw/meshes/Link_2_1.stl" scale="0.001 0.001 0.001"/>
     </geometry>
   </collision>
@@ -89,5 +89,5 @@
     <origin xyz="-0.000321 -0.091983 -0.662215" rpy="0 0 0"/>
     <geometry>
-      <mesh filename="package://melfa_robot/meshes/Link_3_1.stl" scale="0.001 0.001 0.001"/>
+      <mesh filename="package://melfa_assita_ros2_hw/meshes/Link_3_1.stl" scale="0.001 0.001 0.001"/>
     </geometry>
     <material name="silver"/>
@@ -96,5 +96,5 @@
     <origin xyz="-0.000321 -0.091983 -0.662215" rpy="0 0 0"/>
     <geometry>
-      <mesh filename="package://melfa_robot/meshes/Link_3_1.stl" scale="0.001 0.001 0.001"/>
+      <mesh filename="package://melfa_assita_ros2_hw/meshes/Link_3_1.stl" scale="0.001 0.001 0.001"/>
     </geometry>
   </collision>
@@ -109,5 +109,5 @@
     <origin xyz="-0.000488 -0.000483 -0.819715" rpy="0 0 0"/>
     <geometry>
-      <mesh filename="package://melfa_robot/meshes/Link_4_1.stl" scale="0.001 0.001 0.001"/>
+      <mesh filename="package://melfa_assita_ros2_hw/meshes/Link_4_1.stl" scale="0.001 0.001 0.001"/>
     </geometry>
     <material name="silver"/>
@@ -116,5 +116,5 @@
     <origin xyz="-0.000488 -0.000483 -0.819715" rpy="0 0 0"/>
     <geometry>
-      <mesh filename="package://melfa_robot/meshes/Link_4_1.stl" scale="0.001 0.001 0.001"/>
+      <mesh filename="package://melfa_assita_ros2_hw/meshes/Link_4_1.stl" scale="0.001 0.001 0.001"/>
     </geometry>
   </collision>
@@ -129,5 +129,5 @@
     <origin xyz="-0.000488 0.051017 -1.165215" rpy="0 0 0"/>
     <geometry>
-      <mesh filename="package://melfa_robot/meshes/Link_5_1.stl" scale="0.001 0.001 0.001"/>
+      <mesh filename="package://melfa_assita_ros2_hw/meshes/Link_5_1.stl" scale="0.001 0.001 0.001"/>
     </geometry>
     <material name="silver"/>
@@ -136,5 +136,5 @@
     <origin xyz="-0.000488 0.051017 -1.165215" rpy="0 0 0"/>
     <geometry>
-      <mesh filename="package://melfa_robot/meshes/Link_5_1.stl" scale="0.001 0.001 0.001"/>
+      <mesh filename="package://melfa_assita_ros2_hw/meshes/Link_5_1.stl" scale="0.001 0.001 0.001"/>
     </geometry>
   </collision>
@@ -149,5 +149,5 @@
     <origin xyz="-0.000317 -0.001983 -1.271215" rpy="0 0 0"/>
     <geometry>
-      <mesh filename="package://melfa_robot/meshes/Link_6_1.stl" scale="0.001 0.001 0.001"/>
+      <mesh filename="package://melfa_assita_ros2_hw/meshes/Link_6_1.stl" scale="0.001 0.001 0.001"/>
     </geometry>
     <material name="silver"/>
@@ -156,5 +156,5 @@
     <origin xyz="-0.000317 -0.001983 -1.271215" rpy="0 0 0"/>
     <geometry>
-      <mesh filename="package://melfa_robot/meshes/Link_6_1.stl" scale="0.001 0.001 0.001"/>
+      <mesh filename="package://melfa_assita_ros2_hw/meshes/Link_6_1.stl" scale="0.001 0.001 0.001"/>
     </geometry>
   </collision>
