Commit message: Updated the Path Fixed Issure and Gernated the Moveit2 Packet

File: melfa-assista-hardware/description/ros2_control/melfa.ros2_control.xacro (robot description, xacro)
@@ -21,57 +21,55 @@
       </xacro:unless>
       <joint name="joint_1">
+        <param name="initial_value">0.0</param>
         <command_interface name="position">
-          <param name="min">{-(240 * pi)/180}</param>
-          <param name="max">{(240 * pi)/180}</param>
+          <param name="min">-2.62</param>
+          <param name="max">2.62</param>
         </command_interface>
-        <state_interface name="position">
-          <param name="initial_value">0.0</param>
-        </state_interface>
+        <state_interface name="position"/>
       </joint>
       <joint name="joint_2">
+      <param name="initial_value">0.0</param>
         <command_interface name="position">
-          <param name="min">{-(148 * pi)/180}</param>
-          <param name="max">{(148 * pi)/180}</param>
+          <param name="min">-2.58</param>
+          <param name="max">+2.58</param>
         </command_interface>
-        <state_interface name="position">
-          <param name="initial_value">0.0</param>
-        </state_interface>
+         <state_interface name="position"/>
       </joint>
       <joint name="joint_3">
+      <param name="initial_value">1.57</param>
         <command_interface name="position">
-          <param name="min">{-(150 * pi)/180}</param>
-          <param name="max">{(150 * pi)/180}</param>
+          <param name="min">-2.62</param>
+          <param name="max">2.62</param>
         </command_interface>
-        <state_interface name="position">
-          <param name="initial_value">0.0</param>
-        </state_interface>
+         <state_interface name="position"/>
       </joint>
       <joint name="joint_4">
+      <param name="initial_value">0.0</param>
         <command_interface name="position">
-          <param name="min">{-(200 * pi)/180}</param>
-          <param name="max">{(200 * pi)/180}</param>
+          <param name="min">-3.49</param>
+          <param name="max">3.49</param>
         </command_interface>
-        <state_interface name="position">
-          <param name="initial_value">0.0</param>
-        </state_interface>
+         <state_interface name="position"/>
       </joint>
       <joint name="joint_5">
+      <param name="initial_value">1.57</param>
         <command_interface name="position">
-          <param name="min">{-(120 * pi)/180}</param>
-          <param name="max">{(120 * pi)/180}</param>
+          <param name="min">-2.0</param>
+          <param name="max">2.0</param>
         </command_interface>
-        <state_interface name="position">
-          <param name="initial_value">0.0</param>
-        </state_interface>
+         <state_interface name="position"/>
       </joint>
       <joint name="joint_6">
+      <param name="initial_value">0.0</param>
         <command_interface name="position">
-          <param name="min">{-(200 * pi)/180}</param>
-          <param name="max">{(200 * pi)/180}</param>
+          <param name="min">-3.49</param>
+          <param name="max">3.49</param>
         </command_interface>
-        <state_interface name="position">
-          <param name="initial_value">0.0</param>
-        </state_interface>
+         <state_interface name="position"/>
       </joint>
+      <gpio name="Tool">
+        <command_interface name="Tool"/>
+        <state_interface name="Tool"/>
+      </gpio>
     </ros2_control>
   </xacro:macro>

File: melfa-assista-hardware/description/urdf/RV-5AS.urdf.xacro (robot description, xacro)
@@ -170,5 +170,5 @@
   <child link="Link_1_1"/>
   <axis xyz="0.0 0.0 1.0"/>
-  <limit lower="${-(240 * pi)/180}" upper="${(240 * pi)/180}" effort="100" velocity="${(124*pi)/180}"/>
+  <limit lower="${-(240 * pi)/180}" upper="${(240 * pi)/180}" effort="1000" velocity="${(124*pi)/180}"/>
 </joint>
 <joint name="joint_2" type="revolute">
@@ -177,5 +177,5 @@
   <child link="Link_2_1"/>
   <axis xyz="0.0 1.0 -0.0"/>
-  <limit lower="${-(148 * pi)/180}" upper="${(148 * pi)/180}" effort="100" velocity="${(124*pi)/180}"/>
+  <limit lower="${-(148 * pi)/180}" upper="${(148 * pi)/180}" effort="1000" velocity="${(124*pi)/180}"/>
 </joint>
 <joint name="joint_3" type="revolute">
@@ -184,5 +184,5 @@
   <child link="Link_3_1"/>
   <axis xyz="-0.0 1.0 0.0"/>
-  <limit lower="${-(150 * pi)/180}" upper="${(150 * pi)/180}" effort="100" velocity="${(124*pi)/180}"/>
+  <limit lower="${-(150 * pi)/180}" upper="${(150 * pi)/180}" effort="1000" velocity="${(124*pi)/180}"/>
 </joint>
 <joint name="joint_4" type="revolute">
@@ -191,5 +191,5 @@
   <child link="Link_4_1"/>
   <axis xyz="0.0 0.0 1.0"/>
-  <limit lower="${-(200 * pi)/180}" upper="${(200 * pi)/180}" effort="100" velocity="${(124*pi)/180}"/>
+  <limit lower="${-(200 * pi)/180}" upper="${(200 * pi)/180}" effort="1000" velocity="${(124*pi)/180}"/>
 </joint>
 <joint name="joint_5" type="revolute">
@@ -198,5 +198,5 @@
   <child link="Link_5_1"/>
   <axis xyz="0.0 1.0 -0.0"/>
-  <limit lower="${-(120 * pi)/180}" upper="${(120 * pi)/180}" effort="100" velocity="${(356*pi)/180}"/>
+  <limit lower="${-(120 * pi)/180}" upper="${(120 * pi)/180}" effort="1000" velocity="${(356*pi)/180}"/>
 </joint>
 <joint name="joint_6" type="revolute">
@@ -205,5 +205,5 @@
   <child link="Link_6_1"/>
   <axis xyz="0.0 0.0 1.0"/>
-  <limit lower="${-(200 * pi)/180}" upper="${(200 * pi)/180}" effort="100" velocity="${(360*pi)/180}"/>
+  <limit lower="${-(200 * pi)/180}" upper="${(200 * pi)/180}" effort="1000" velocity="${(360*pi)/180}"/>
 </joint>
 </robot>

Commit message: Fixed Build Error

File: melfa-assista-hardware/description/ros2_control/melfa.ros2_control.xacro (robot description, xacro)
@@ -15,5 +15,5 @@
           </xacro:if>
           <xacro:unless value="${use_fake_hardware}">
-            <plugin>melfa_assita_ros2_hw/MelfaHW</plugin>
+            <plugin>melfa-assista-hardware/MelfaHW</plugin>
             <param name="robot_ip">${robot_ip}</param>
           </xacro:unless>

File: melfa-assista-hardware/description/urdf/RV-5AS.urdf.xacro (robot description, xacro)
@@ -5,7 +5,7 @@
 <xacro:arg name="use_fake_hardware" default="true" />
 <xacro:arg name="robot_ip" default="127.0.0.1" />
-<xacro:include filename="$(find melfa_assita_ros2_hw)/urdf/materials.xacro" />
-<xacro:include filename="$(find melfa_assita_ros2_hw)/urdf/RV-5AS.gazebo" />
-<xacro:include filename="$(find melfa_assita_ros2_hw)/ros2_control/melfa.ros2_control.xacro" />
+<xacro:include filename="$(find melfa-assista-hardware)/urdf/materials.xacro" />
+<xacro:include filename="$(find melfa-assista-hardware)/urdf/RV-5AS.gazebo" />
+<xacro:include filename="$(find melfa-assista-hardware)/ros2_control/melfa.ros2_control.xacro" />
 <!-- Enable Gazebo Plugins -->
   <gazebo>
@@ -13,5 +13,5 @@
       <!-- <robot_param>robot_description</robot_param>
       <robot_param_node>robot_state_publisher</robot_param_node> -->
-      <parameters>$(find melfa_assita_ros2_hw)/config/melfa_controller.yaml</parameters>
+      <parameters>$(find melfa-assista-hardware)/config/melfa_controller.yaml</parameters>
     </plugin>
   </gazebo>
@@ -28,5 +28,5 @@
     <origin xyz="0 0 0" rpy="0 0 0"/>
     <geometry>
-      <mesh filename="package://melfa_assita_ros2_hw/meshes/base_link.stl" scale="0.001 0.001 0.001"/>
+      <mesh filename="package://melfa-assista-hardware/meshes/base_link.stl" scale="0.001 0.001 0.001"/>
       <cylinder radius="0.5" length="1.0"/>
     </geometry>
@@ -36,5 +36,5 @@
     <origin xyz="0 0 0" rpy="0 0 0"/>
     <geometry>
-      <mesh filename="package://melfa_assita_ros2_hw/meshes/base_link.stl" scale="0.001 0.001 0.001"/>
+      <mesh filename="package://melfa-assista-hardware/meshes/base_link.stl" scale="0.001 0.001 0.001"/>
     </geometry>
   </collision>
@@ -49,5 +49,5 @@
     <origin xyz="-0.000321 -0.000483 -0.169215" rpy="0 0 0"/>
     <geometry>
-      <mesh filename="package://melfa_assita_ros2_hw/meshes/Link_1_1.stl" scale="0.001 0.001 0.001"/>
+      <mesh filename="package://melfa-assista-hardware/meshes/Link_1_1.stl" scale="0.001 0.001 0.001"/>
     </geometry>
     <material name="silver"/>
@@ -56,5 +56,5 @@
     <origin xyz="-0.000321 -0.000483 -0.169215" rpy="0 0 0"/>
     <geometry>
-      <mesh filename="package://melfa_assita_ros2_hw/meshes/Link_1_1.stl" scale="0.001 0.001 0.001"/>
+      <mesh filename="package://melfa-assista-hardware/meshes/Link_1_1.stl" scale="0.001 0.001 0.001"/>
     </geometry>
   </collision>
@@ -69,5 +69,5 @@
     <origin xyz="-0.000321 -0.091983 -0.252215" rpy="0 0 0"/>
     <geometry>
-      <mesh filename="package://melfa_assita_ros2_hw/meshes/Link_2_1.stl" scale="0.001 0.001 0.001"/>
+      <mesh filename="package://melfa-assista-hardware/meshes/Link_2_1.stl" scale="0.001 0.001 0.001"/>
     </geometry>
     <material name="silver"/>
@@ -76,5 +76,5 @@
     <origin xyz="-0.000321 -0.091983 -0.252215" rpy="0 0 0"/>
     <geometry>
-      <mesh filename="package://melfa_assita_ros2_hw/meshes/Link_2_1.stl" scale="0.001 0.001 0.001"/>
+      <mesh filename="package://melfa-assista-hardware/meshes/Link_2_1.stl" scale="0.001 0.001 0.001"/>
     </geometry>
   </collision>
@@ -89,5 +89,5 @@
     <origin xyz="-0.000321 -0.091983 -0.662215" rpy="0 0 0"/>
     <geometry>
-      <mesh filename="package://melfa_assita_ros2_hw/meshes/Link_3_1.stl" scale="0.001 0.001 0.001"/>
+      <mesh filename="package://melfa-assista-hardware/meshes/Link_3_1.stl" scale="0.001 0.001 0.001"/>
     </geometry>
     <material name="silver"/>
@@ -96,5 +96,5 @@
     <origin xyz="-0.000321 -0.091983 -0.662215" rpy="0 0 0"/>
     <geometry>
-      <mesh filename="package://melfa_assita_ros2_hw/meshes/Link_3_1.stl" scale="0.001 0.001 0.001"/>
+      <mesh filename="package://melfa-assista-hardware/meshes/Link_3_1.stl" scale="0.001 0.001 0.001"/>
     </geometry>
   </collision>
@@ -109,5 +109,5 @@
     <origin xyz="-0.000488 -0.000483 -0.819715" rpy="0 0 0"/>
     <geometry>
-      <mesh filename="package://melfa_assita_ros2_hw/meshes/Link_4_1.stl" scale="0.001 0.001 0.001"/>
+      <mesh filename="package://melfa-assista-hardware/meshes/Link_4_1.stl" scale="0.001 0.001 0.001"/>
     </geometry>
     <material name="silver"/>
@@ -116,5 +116,5 @@
     <origin xyz="-0.000488 -0.000483 -0.819715" rpy="0 0 0"/>
     <geometry>
-      <mesh filename="package://melfa_assita_ros2_hw/meshes/Link_4_1.stl" scale="0.001 0.001 0.001"/>
+      <mesh filename="package://melfa-assista-hardware/meshes/Link_4_1.stl" scale="0.001 0.001 0.001"/>
     </geometry>
   </collision>
@@ -129,5 +129,5 @@
     <origin xyz="-0.000488 0.051017 -1.165215" rpy="0 0 0"/>
     <geometry>
-      <mesh filename="package://melfa_assita_ros2_hw/meshes/Link_5_1.stl" scale="0.001 0.001 0.001"/>
+      <mesh filename="package://melfa-assista-hardware/meshes/Link_5_1.stl" scale="0.001 0.001 0.001"/>
     </geometry>
     <material name="silver"/>
@@ -136,5 +136,5 @@
     <origin xyz="-0.000488 0.051017 -1.165215" rpy="0 0 0"/>
     <geometry>
-      <mesh filename="package://melfa_assita_ros2_hw/meshes/Link_5_1.stl" scale="0.001 0.001 0.001"/>
+      <mesh filename="package://melfa-assista-hardware/meshes/Link_5_1.stl" scale="0.001 0.001 0.001"/>
     </geometry>
   </collision>
@@ -149,5 +149,5 @@
     <origin xyz="-0.000317 -0.001983 -1.271215" rpy="0 0 0"/>
     <geometry>
-      <mesh filename="package://melfa_assita_ros2_hw/meshes/Link_6_1.stl" scale="0.001 0.001 0.001"/>
+      <mesh filename="package://melfa-assista-hardware/meshes/Link_6_1.stl" scale="0.001 0.001 0.001"/>
     </geometry>
     <material name="silver"/>
@@ -156,5 +156,5 @@
     <origin xyz="-0.000317 -0.001983 -1.271215" rpy="0 0 0"/>
     <geometry>
-      <mesh filename="package://melfa_assita_ros2_hw/meshes/Link_6_1.stl" scale="0.001 0.001 0.001"/>
+      <mesh filename="package://melfa-assista-hardware/meshes/Link_6_1.stl" scale="0.001 0.001 0.001"/>
     </geometry>
   </collision>

File: melfa-assista-moveit/config/Assista.urdf.xacro (robot description, xacro)
@@ -3,5 +3,5 @@
     <xacro:arg name="initial_positions_file" default="initial_positions.yaml" />
     <!-- Import Assista urdf file -->
-    <xacro:include filename="$(find melfa_assita_ros2_hw)/urdf/RV-5AS.urdf.xacro" />
+    <xacro:include filename="$(find melfa-assista-hardware)/urdf/RV-5AS.urdf.xacro" />
     <!-- Import control_xacro -->
     <xacro:include filename="Assista.ros2_control.xacro" />
