Commit message: Fixed Error with Pluglib

File: melfa-assista-moveit/config/Assista.urdf.xacro (robot description, xacro)
@@ -3,5 +3,5 @@
     <xacro:arg name="initial_positions_file" default="initial_positions.yaml" />
     <!-- Import Assista urdf file -->
-    <xacro:include filename="$(find melfa-assista-hardware)/urdf/RV-5AS.urdf.xacro" />
+    <xacro:include filename="$(find melfa_assista_hardware)/urdf/RV-5AS.urdf.xacro" />
     <!-- Import control_xacro -->
     <xacro:include filename="Assista.ros2_control.xacro" />

File: melfa_assista_hardware/description/ros2_control/melfa.ros2_control.xacro (robot description, xacro)
@@ -15,5 +15,5 @@
           </xacro:if>
           <xacro:unless value="${use_fake_hardware}">
-            <plugin>melfa-assista-hardware/MelfaHW</plugin>
+            <plugin>melfa_assista_hardware/MelfaHW</plugin>
             <param name="robot_ip">${robot_ip}</param>
           </xacro:unless>
@@ -68,8 +68,4 @@
          <state_interface name="position"/>
       </joint>
-      <gpio name="Tool">
-        <command_interface name="Tool"/>
-        <state_interface name="Tool"/>
-      </gpio>
     </ros2_control>
   </xacro:macro>

File: melfa_assista_hardware/description/urdf/RV-5AS.urdf.xacro (robot description, xacro)
@@ -5,7 +5,7 @@
 <xacro:arg name="use_fake_hardware" default="true" />
 <xacro:arg name="robot_ip" default="127.0.0.1" />
-<xacro:include filename="$(find melfa-assista-hardware)/urdf/materials.xacro" />
-<xacro:include filename="$(find melfa-assista-hardware)/urdf/RV-5AS.gazebo" />
-<xacro:include filename="$(find melfa-assista-hardware)/ros2_control/melfa.ros2_control.xacro" />
+<xacro:include filename="$(find melfa_assista_hardware)/urdf/materials.xacro" />
+<xacro:include filename="$(find melfa_assista_hardware)/urdf/RV-5AS.gazebo" />
+<xacro:include filename="$(find melfa_assista_hardware)/ros2_control/melfa.ros2_control.xacro" />
 <!-- Enable Gazebo Plugins -->
   <gazebo>
@@ -13,5 +13,5 @@
       <!-- <robot_param>robot_description</robot_param>
       <robot_param_node>robot_state_publisher</robot_param_node> -->
-      <parameters>$(find melfa-assista-hardware)/config/melfa_controller.yaml</parameters>
+      <parameters>$(find melfa_assista_hardware)/config/melfa_controller.yaml</parameters>
     </plugin>
   </gazebo>
@@ -28,5 +28,5 @@
     <origin xyz="0 0 0" rpy="0 0 0"/>
     <geometry>
-      <mesh filename="package://melfa-assista-hardware/meshes/base_link.stl" scale="0.001 0.001 0.001"/>
+      <mesh filename="package://melfa_assista_hardware/meshes/base_link.stl" scale="0.001 0.001 0.001"/>
       <cylinder radius="0.5" length="1.0"/>
     </geometry>
@@ -36,5 +36,5 @@
     <origin xyz="0 0 0" rpy="0 0 0"/>
     <geometry>
-      <mesh filename="package://melfa-assista-hardware/meshes/base_link.stl" scale="0.001 0.001 0.001"/>
+      <mesh filename="package://melfa_assista_hardware/meshes/base_link.stl" scale="0.001 0.001 0.001"/>
     </geometry>
   </collision>
@@ -49,5 +49,5 @@
     <origin xyz="-0.000321 -0.000483 -0.169215" rpy="0 0 0"/>
     <geometry>
-      <mesh filename="package://melfa-assista-hardware/meshes/Link_1_1.stl" scale="0.001 0.001 0.001"/>
+      <mesh filename="package://melfa_assista_hardware/meshes/Link_1_1.stl" scale="0.001 0.001 0.001"/>
     </geometry>
     <material name="silver"/>
@@ -56,5 +56,5 @@
     <origin xyz="-0.000321 -0.000483 -0.169215" rpy="0 0 0"/>
     <geometry>
-      <mesh filename="package://melfa-assista-hardware/meshes/Link_1_1.stl" scale="0.001 0.001 0.001"/>
+      <mesh filename="package://melfa_assista_hardware/meshes/Link_1_1.stl" scale="0.001 0.001 0.001"/>
     </geometry>
   </collision>
@@ -69,5 +69,5 @@
     <origin xyz="-0.000321 -0.091983 -0.252215" rpy="0 0 0"/>
     <geometry>
-      <mesh filename="package://melfa-assista-hardware/meshes/Link_2_1.stl" scale="0.001 0.001 0.001"/>
+      <mesh filename="package://melfa_assista_hardware/meshes/Link_2_1.stl" scale="0.001 0.001 0.001"/>
     </geometry>
     <material name="silver"/>
@@ -76,5 +76,5 @@
     <origin xyz="-0.000321 -0.091983 -0.252215" rpy="0 0 0"/>
     <geometry>
-      <mesh filename="package://melfa-assista-hardware/meshes/Link_2_1.stl" scale="0.001 0.001 0.001"/>
+      <mesh filename="package://melfa_assista_hardware/meshes/Link_2_1.stl" scale="0.001 0.001 0.001"/>
     </geometry>
   </collision>
@@ -89,5 +89,5 @@
     <origin xyz="-0.000321 -0.091983 -0.662215" rpy="0 0 0"/>
     <geometry>
-      <mesh filename="package://melfa-assista-hardware/meshes/Link_3_1.stl" scale="0.001 0.001 0.001"/>
+      <mesh filename="package://melfa_assista_hardware/meshes/Link_3_1.stl" scale="0.001 0.001 0.001"/>
     </geometry>
     <material name="silver"/>
@@ -96,5 +96,5 @@
     <origin xyz="-0.000321 -0.091983 -0.662215" rpy="0 0 0"/>
     <geometry>
-      <mesh filename="package://melfa-assista-hardware/meshes/Link_3_1.stl" scale="0.001 0.001 0.001"/>
+      <mesh filename="package://melfa_assista_hardware/meshes/Link_3_1.stl" scale="0.001 0.001 0.001"/>
     </geometry>
   </collision>
@@ -109,5 +109,5 @@
     <origin xyz="-0.000488 -0.000483 -0.819715" rpy="0 0 0"/>
     <geometry>
-      <mesh filename="package://melfa-assista-hardware/meshes/Link_4_1.stl" scale="0.001 0.001 0.001"/>
+      <mesh filename="package://melfa_assista_hardware/meshes/Link_4_1.stl" scale="0.001 0.001 0.001"/>
     </geometry>
     <material name="silver"/>
@@ -116,5 +116,5 @@
     <origin xyz="-0.000488 -0.000483 -0.819715" rpy="0 0 0"/>
     <geometry>
-      <mesh filename="package://melfa-assista-hardware/meshes/Link_4_1.stl" scale="0.001 0.001 0.001"/>
+      <mesh filename="package://melfa_assista_hardware/meshes/Link_4_1.stl" scale="0.001 0.001 0.001"/>
     </geometry>
   </collision>
@@ -129,5 +129,5 @@
     <origin xyz="-0.000488 0.051017 -1.165215" rpy="0 0 0"/>
     <geometry>
-      <mesh filename="package://melfa-assista-hardware/meshes/Link_5_1.stl" scale="0.001 0.001 0.001"/>
+      <mesh filename="package://melfa_assista_hardware/meshes/Link_5_1.stl" scale="0.001 0.001 0.001"/>
     </geometry>
     <material name="silver"/>
@@ -136,5 +136,5 @@
     <origin xyz="-0.000488 0.051017 -1.165215" rpy="0 0 0"/>
     <geometry>
-      <mesh filename="package://melfa-assista-hardware/meshes/Link_5_1.stl" scale="0.001 0.001 0.001"/>
+      <mesh filename="package://melfa_assista_hardware/meshes/Link_5_1.stl" scale="0.001 0.001 0.001"/>
     </geometry>
   </collision>
@@ -149,5 +149,5 @@
     <origin xyz="-0.000317 -0.001983 -1.271215" rpy="0 0 0"/>
     <geometry>
-      <mesh filename="package://melfa-assista-hardware/meshes/Link_6_1.stl" scale="0.001 0.001 0.001"/>
+      <mesh filename="package://melfa_assista_hardware/meshes/Link_6_1.stl" scale="0.001 0.001 0.001"/>
     </geometry>
     <material name="silver"/>
@@ -156,5 +156,5 @@
     <origin xyz="-0.000317 -0.001983 -1.271215" rpy="0 0 0"/>
     <geometry>
-      <mesh filename="package://melfa-assista-hardware/meshes/Link_6_1.stl" scale="0.001 0.001 0.001"/>
+      <mesh filename="package://melfa_assista_hardware/meshes/Link_6_1.stl" scale="0.001 0.001 0.001"/>
     </geometry>
   </collision>
