Commit message: Added the Feature to Close and Open a Hand on Port 1

File: melfa_assista_hardware/description/ros2_control/melfa.ros2_control.xacro (robot description, xacro)
@@ -1,6 +1,7 @@
 <?xml version="1.0"?>
 <robot xmlns:xacro="http://www.ros.org/wiki/xacro">
-  <xacro:macro name="melfa_ros2_control" params="name robot_ip use_sim:=^|false use_fake_hardware:=^|true">
-    <ros2_control name="${name}" type="system" >
+  <xacro:macro name="melfa_ros2_control"
+    params="name robot_ip use_sim:=^|false use_fake_hardware:=^|true">
+    <ros2_control name="${name}" type="system">
       <xacro:if value="$(arg use_sim)">
         <hardware>
@@ -26,46 +27,55 @@
           <param name="max">2.62</param>
         </command_interface>
-        <state_interface name="position"/>
+        <state_interface name="position" />
       </joint>
       <joint name="joint_2">
-      <param name="initial_value">0.0</param>
+        <param name="initial_value">0.0</param>
         <command_interface name="position">
           <param name="min">-2.58</param>
           <param name="max">+2.58</param>
         </command_interface>
-         <state_interface name="position"/>
+        <state_interface name="position" />
       </joint>
       <joint name="joint_3">
-      <param name="initial_value">1.57</param>
+        <param name="initial_value">1.57</param>
         <command_interface name="position">
           <param name="min">-2.62</param>
           <param name="max">2.62</param>
         </command_interface>
-         <state_interface name="position"/>
+        <state_interface name="position" />
       </joint>
       <joint name="joint_4">
-      <param name="initial_value">0.0</param>
+        <param name="initial_value">0.0</param>
         <command_interface name="position">
           <param name="min">-3.49</param>
           <param name="max">3.49</param>
         </command_interface>
-         <state_interface name="position"/>
+        <state_interface name="position" />
       </joint>
       <joint name="joint_5">
-      <param name="initial_value">1.57</param>
+        <param name="initial_value">1.57</param>
         <command_interface name="position">
           <param name="min">-2.0</param>
           <param name="max">2.0</param>
         </command_interface>
-         <state_interface name="position"/>
+        <state_interface name="position" />
       </joint>
       <joint name="joint_6">
-      <param name="initial_value">0.0</param>
+        <param name="initial_value">0.0</param>
         <command_interface name="position">
           <param name="min">-3.49</param>
           <param name="max">3.49</param>
         </command_interface>
-         <state_interface name="position"/>
+        <state_interface name="position" />
       </joint>
+      <!-- from https://github.com/ros-controls/ros2_control/blob/f58d4072dbd1c3fd4e1f64cd10a19a2b60f59049/ros2_control_test_assets/include/ros2_control_test_assets/components_urdfs.hpp#L344 -->
+      <gpio name="tool_flansch">
+        <command_interface name="coact">
+          <param name="initial_value">1.0</param>
+        </command_interface>
+        <state_interface name="coact" >
+          <param name="initial_value">1.0</param>
+        </state_interface>
+      </gpio>
     </ros2_control>
   </xacro:macro>
