Commit message: Added the Moveit Config

File: melfa_assista_hardware/description/urdf/RV-5AS.urdf.xacro (robot description, xacro)
@@ -7,8 +7,9 @@
 <xacro:include filename="$(find melfa_assista_hardware)/urdf/materials.xacro" />
 <xacro:include filename="$(find melfa_assista_hardware)/urdf/RV-5AS.gazebo" />
+<xacro:include filename="$(find melfa_assista_hardware)/urdf/Co-Act.xacro" />
 <xacro:include filename="$(find melfa_assista_hardware)/ros2_control/melfa.ros2_control.xacro" />
 <!-- Enable Gazebo Plugins -->
   <gazebo>
-    <plugin filename="libgazebo_ros2_control.so" name="gazebo_ros2_control">
+    <plugin filename="libgazebo_ros2_control.so" name="gazebo_ros2_control.">
       <!-- <robot_param>robot_description</robot_param>
       <robot_param_node>robot_state_publisher</robot_param_node> -->
@@ -207,3 +208,9 @@
   <limit lower="${-(200 * pi)/180}" upper="${(200 * pi)/180}" effort="1000" velocity="${(360*pi)/180}"/>
 </joint>
+<!-- Tool Joint Connection to the Robot -->
+<joint name="joint_tool_robot" type="fixed">
+  <origin xyz="0.0 0.0 0.0" rpy="-${(pi/2)} 0.0 ${(pi/2)}"/>
+  <parent link="Link_6_1"/>
+  <child link="base_coact_link"/>
+</joint>
 </robot>

Commit message: Added the Camera to the Model and added some Errors Managment to the Hardware File

File: melfa_assista_hardware/description/urdf/RV-5AS.urdf.xacro (robot description, xacro)
@@ -7,5 +7,5 @@
 <xacro:include filename="$(find melfa_assista_hardware)/urdf/materials.xacro" />
 <xacro:include filename="$(find melfa_assista_hardware)/urdf/RV-5AS.gazebo" />
-<xacro:include filename="$(find melfa_assista_hardware)/urdf/Co-Act.xacro" />
+<xacro:include filename="$(find melfa_assista_hardware)/urdf/Coact_w_Camera.xacro" />
 <xacro:include filename="$(find melfa_assista_hardware)/ros2_control/melfa.ros2_control.xacro" />
 <!-- Enable Gazebo Plugins -->
@@ -210,7 +210,7 @@
 <!-- Tool Joint Connection to the Robot -->
 <joint name="joint_tool_robot" type="fixed">
-  <origin xyz="0.0 0.0 0.0" rpy="-${(pi/2)} 0.0 ${(pi/2)}"/>
+  <origin xyz="0.0 0.0 0.01" rpy="-${(pi/2)} 0.0 ${(pi/2)}"/>
   <parent link="Link_6_1"/>
-  <child link="base_coact_link"/>
+  <child link="coact_base_link"/>
 </joint>
 </robot>
