Commit message: Xacro Files Updated Split Camera und Tool

File: melfa_assista_hardware/description/urdf/Coact_Schunk.xacro (robot description, xacro)
@@ -3,6 +3,5 @@
      Commit Version: 1.6.0-4-g7f85cfe  Build Version: 1.6.7995.38578
      For more information, please see http://wiki.ros.org/sw_urdf_exporter -->
-<robot
-  name="Coact_wCamera">
+  <robot xmlns:xacro="http://www.ros.org/wiki/xacro">
   <link
     name="coact_base_link">
@@ -151,8 +150,8 @@
       xyz="1 0 0" />
     <limit
-      lower="0"
+      lower="0.0"
       upper="0.006"
       effort="200"
-      velocity="1" />
+      velocity="1.0" />
   </joint>
   <link
@@ -262,8 +261,8 @@
       xyz="1 0 0" />
     <limit
-      lower="0"
+      lower="0.0"
       upper="0.006"
       effort="200"
-      velocity="1" />
+      velocity="1.0" />
     <mimic
       joint="joint_hand_left"
@@ -324,109 +323,3 @@
       xyz="0 0 0" />
   </joint>
-  <link
-    name="camea_adapter_link">
-    <inertial>
-      <origin
-        xyz="6.8987E-05 6.8987E-05 0.0086472"
-        rpy="0 0 0" />
-      <mass
-        value="0.11061" />
-      <inertia
-        ixx="0.00011703"
-        ixy="-7.4547E-10"
-        ixz="3.2264E-07"
-        iyy="0.00012118"
-        iyz="-6.0814E-08"
-        izz="2.26E-05" />
-    </inertial>
-    <visual>
-      <origin
-        xyz="0 0 0"
-        rpy="0 0 0" />
-      <geometry>
-        <mesh
-          filename="package://melfa_assista_hardware/meshes/camea_adapter_link.STL" />
-      </geometry>
-      <material
-        name="">
-        <color
-          rgba="1 1 1 1" />
-      </material>
-    </visual>
-    <collision>
-      <origin
-        xyz="0 0 0"
-        rpy="0 0 0" />
-      <geometry>
-        <mesh
-          filename="package://melfa_assista_hardware/meshes/camea_adapter_link.STL" />
-      </geometry>
-    </collision>
-  </link>
-  <joint
-    name="joint_camera_adapter"
-    type="fixed">
-    <origin
-      xyz="-0.00275 -0.0425 -0.04425"
-      rpy="-1.5708 0 0" />
-    <parent
-      link="coact_base_link" />
-    <child
-      link="camea_adapter_link" />
-    <axis
-      xyz="0 0 0" />
-  </joint>
-  <link
-    name="camera_link">
-    <inertial>
-      <origin
-        xyz="6.8987E-05 8.2543E-06 0.0086472"
-        rpy="0 0 0" />
-      <mass
-        value="0.11061" />
-      <inertia
-        ixx="0.00011703"
-        ixy="-7.4547E-10"
-        ixz="3.2264E-07"
-        iyy="0.00012118"
-        iyz="-6.0814E-08"
-        izz="2.26E-05" />
-    </inertial>
-    <visual>
-      <origin
-        xyz="0 0 0"
-        rpy="0 0 0" />
-      <geometry>
-        <mesh
-          filename="package://melfa_assista_hardware/meshes/camera_link.STL" />
-      </geometry>
-      <material
-        name="">
-        <color
-          rgba="0.50196 0.50196 0.50196 1" />
-      </material>
-    </visual>
-    <collision>
-      <origin
-        xyz="0 0 0"
-        rpy="0 0 0" />
-      <geometry>
-        <mesh
-          filename="package://melfa_assista_hardware/meshes/camera_link.STL" />
-      </geometry>
-    </collision>
-  </link>
-  <joint
-    name="joint_camera"
-    type="fixed">
-    <origin
-      xyz="0 0.027 -0.0185"
-      rpy="3.1416 0 3.1416" />
-    <parent
-      link="camea_adapter_link" />
-    <child
-      link="camera_link" />
-    <axis
-      xyz="0 0 0" />
-  </joint>
 </robot>

File: melfa_assista_hardware/description/urdf/RV-5AS.urdf.xacro (robot description, xacro)
@@ -7,11 +7,12 @@
 <xacro:include filename="$(find melfa_assista_hardware)/urdf/materials.xacro" />
 <xacro:include filename="$(find melfa_assista_hardware)/urdf/RV-5AS.gazebo" />
-<xacro:include filename="$(find melfa_assista_hardware)/urdf/Coact_w_Camera.xacro" />
+<xacro:include filename="$(find melfa_assista_hardware)/urdf/Coact_Schunk.xacro" />
+<xacro:include filename="$(find melfa_assista_hardware)/urdf/Camera.xacro" />
 <xacro:include filename="$(find melfa_assista_hardware)/ros2_control/melfa.ros2_control.xacro" />
 <!-- Enable Gazebo Plugins -->
   <gazebo>
-    <plugin filename="libgazebo_ros2_control.so" name="gazebo_ros2_control.">
-      <!-- <robot_param>robot_description</robot_param>
-      <robot_param_node>robot_state_publisher</robot_param_node> -->
+    <plugin filename="libgazebo_ros2_control.so" name="gazebo_ros2_control.so">
+      <robot_param>robot_description</robot_param>
+      <robot_param_node>robot_state_publisher</robot_param_node>
       <parameters>$(find melfa_assista_hardware)/config/melfa_controller.yaml</parameters>
     </plugin>
