Commit message: Added Support for Gazebo and Camera

File: melfa_assista_hardware/description/urdf/assista_robot.xacro (robot description, xacro)
@@ -1,22 +1,4 @@
 <?xml version="1.0" ?>
-<robot name="Assista" xmlns:xacro="http://www.ros.org/wiki/xacro">
-<!-- Enable setting arguments from the launch file -->
-<xacro:arg name="use_sim" default="false" />
-<xacro:arg name="use_fake_hardware" default="true" />
-<xacro:arg name="robot_ip" default="127.0.0.1" />
-<xacro:include filename="$(find melfa_assista_hardware)/urdf/materials.xacro" />
-<xacro:include filename="$(find melfa_assista_hardware)/urdf/RV-5AS.gazebo" />
-<xacro:include filename="$(find melfa_assista_hardware)/urdf/Coact_Schunk.xacro" />
-<xacro:include filename="$(find melfa_assista_hardware)/urdf/Camera.xacro" />
-<xacro:include filename="$(find melfa_assista_hardware)/ros2_control/melfa.ros2_control.xacro" />
-<!-- Enable Gazebo Plugins -->
-  <gazebo>
-    <plugin filename="libgazebo_ros2_control.so" name="gazebo_ros2_control.so">
-      <robot_param>robot_description</robot_param>
-      <robot_param_node>robot_state_publisher</robot_param_node>
-      <parameters>$(find melfa_assista_hardware)/config/melfa_controller.yaml</parameters>
-    </plugin>
-  </gazebo>
-<xacro:melfa_ros2_control name="melfaHW" robot_ip="$(arg robot_ip)"  use_sim="$(arg use_sim)" use_fake_hardware="$(arg use_fake_hardware)" />
+<robot xmlns:xacro="http://www.ros.org/wiki/xacro">
 <link name="world">
 </link>
@@ -30,5 +12,5 @@
     <origin xyz="0 0 0" rpy="0 0 0"/>
     <geometry>
-      <mesh filename="package://melfa_assista_hardware/meshes/base_link.stl" scale="0.001 0.001 0.001"/>
+      <mesh filename="file://$(find melfa_assista_hardware)/meshes/base_link.STL" scale="0.001 0.001 0.001"/>
       <cylinder radius="0.5" length="1.0"/>
     </geometry>
@@ -38,5 +20,5 @@
     <origin xyz="0 0 0" rpy="0 0 0"/>
     <geometry>
-      <mesh filename="package://melfa_assista_hardware/meshes/base_link.stl" scale="0.001 0.001 0.001"/>
+      <mesh filename="file://$(find melfa_assista_hardware)/meshes/base_link.STL" scale="0.001 0.001 0.001"/>
     </geometry>
   </collision>
@@ -51,5 +33,5 @@
     <origin xyz="-0.000321 -0.000483 -0.169215" rpy="0 0 0"/>
     <geometry>
-      <mesh filename="package://melfa_assista_hardware/meshes/Link_1_1.stl" scale="0.001 0.001 0.001"/>
+      <mesh filename="file://$(find melfa_assista_hardware)/meshes/Link_1_1.stl" scale="0.001 0.001 0.001"/>
     </geometry>
     <material name="silver"/>
@@ -58,5 +40,5 @@
     <origin xyz="-0.000321 -0.000483 -0.169215" rpy="0 0 0"/>
     <geometry>
-      <mesh filename="package://melfa_assista_hardware/meshes/Link_1_1.stl" scale="0.001 0.001 0.001"/>
+      <mesh filename="file://$(find melfa_assista_hardware)/meshes/Link_1_1.stl" scale="0.001 0.001 0.001"/>
     </geometry>
   </collision>
@@ -71,5 +53,5 @@
     <origin xyz="-0.000321 -0.091983 -0.252215" rpy="0 0 0"/>
     <geometry>
-      <mesh filename="package://melfa_assista_hardware/meshes/Link_2_1.stl" scale="0.001 0.001 0.001"/>
+      <mesh filename="file://$(find melfa_assista_hardware)/meshes/Link_2_1.stl" scale="0.001 0.001 0.001"/>
     </geometry>
     <material name="silver"/>
@@ -78,5 +60,5 @@
     <origin xyz="-0.000321 -0.091983 -0.252215" rpy="0 0 0"/>
     <geometry>
-      <mesh filename="package://melfa_assista_hardware/meshes/Link_2_1.stl" scale="0.001 0.001 0.001"/>
+      <mesh filename="file://$(find melfa_assista_hardware)/meshes/Link_2_1.stl" scale="0.001 0.001 0.001"/>
     </geometry>
   </collision>
@@ -91,5 +73,5 @@
     <origin xyz="-0.000321 -0.091983 -0.662215" rpy="0 0 0"/>
     <geometry>
-      <mesh filename="package://melfa_assista_hardware/meshes/Link_3_1.stl" scale="0.001 0.001 0.001"/>
+      <mesh filename="file://$(find melfa_assista_hardware)/meshes/Link_3_1.stl" scale="0.001 0.001 0.001"/>
     </geometry>
     <material name="silver"/>
@@ -98,5 +80,5 @@
     <origin xyz="-0.000321 -0.091983 -0.662215" rpy="0 0 0"/>
     <geometry>
-      <mesh filename="package://melfa_assista_hardware/meshes/Link_3_1.stl" scale="0.001 0.001 0.001"/>
+      <mesh filename="file://$(find melfa_assista_hardware)/meshes/Link_3_1.stl" scale="0.001 0.001 0.001"/>
     </geometry>
   </collision>
@@ -111,5 +93,5 @@
     <origin xyz="-0.000488 -0.000483 -0.819715" rpy="0 0 0"/>
     <geometry>
-      <mesh filename="package://melfa_assista_hardware/meshes/Link_4_1.stl" scale="0.001 0.001 0.001"/>
+      <mesh filename="file://$(find melfa_assista_hardware)/meshes/Link_4_1.stl" scale="0.001 0.001 0.001"/>
     </geometry>
     <material name="silver"/>
@@ -118,5 +100,5 @@
     <origin xyz="-0.000488 -0.000483 -0.819715" rpy="0 0 0"/>
     <geometry>
-      <mesh filename="package://melfa_assista_hardware/meshes/Link_4_1.stl" scale="0.001 0.001 0.001"/>
+      <mesh filename="file://$(find melfa_assista_hardware)/meshes/Link_4_1.stl" scale="0.001 0.001 0.001"/>
     </geometry>
   </collision>
@@ -131,5 +113,5 @@
     <origin xyz="-0.000488 0.051017 -1.165215" rpy="0 0 0"/>
     <geometry>
-      <mesh filename="package://melfa_assista_hardware/meshes/Link_5_1.stl" scale="0.001 0.001 0.001"/>
+      <mesh filename="file://$(find melfa_assista_hardware)/meshes/Link_5_1.stl" scale="0.001 0.001 0.001"/>
     </geometry>
     <material name="silver"/>
@@ -138,5 +120,5 @@
     <origin xyz="-0.000488 0.051017 -1.165215" rpy="0 0 0"/>
     <geometry>
-      <mesh filename="package://melfa_assista_hardware/meshes/Link_5_1.stl" scale="0.001 0.001 0.001"/>
+      <mesh filename="file://$(find melfa_assista_hardware)/meshes/Link_5_1.stl" scale="0.001 0.001 0.001"/>
     </geometry>
   </collision>
@@ -151,5 +133,5 @@
     <origin xyz="-0.000317 -0.001983 -1.271215" rpy="0 0 0"/>
     <geometry>
-      <mesh filename="package://melfa_assista_hardware/meshes/Link_6_1.stl" scale="0.001 0.001 0.001"/>
+      <mesh filename="file://$(find melfa_assista_hardware)/meshes/Link_6_1.stl" scale="0.001 0.001 0.001"/>
     </geometry>
     <material name="silver"/>
@@ -158,5 +140,5 @@
     <origin xyz="-0.000317 -0.001983 -1.271215" rpy="0 0 0"/>
     <geometry>
-      <mesh filename="package://melfa_assista_hardware/meshes/Link_6_1.stl" scale="0.001 0.001 0.001"/>
+      <mesh filename="file://$(find melfa_assista_hardware)/meshes/Link_6_1.stl" scale="0.001 0.001 0.001"/>
     </geometry>
   </collision>
@@ -209,9 +191,3 @@
   <limit lower="${-(200 * pi)/180}" upper="${(200 * pi)/180}" effort="1000" velocity="${(360*pi)/180}"/>
 </joint>
-<!-- Tool Joint Connection to the Robot -->
-<joint name="joint_tool_robot" type="fixed">
-  <origin xyz="0.0 0.0 0.01" rpy="-${(pi/2)} 0.0 ${(pi/2)}"/>
-  <parent link="Link_6_1"/>
-  <child link="coact_base_link"/>
-</joint>
 </robot>

File: melfa_assista_hardware/description/urdf/camera.xacro (robot description, xacro)
@@ -11,5 +11,5 @@
             <origin xyz="0 0 0" rpy="0 0 0" />
             <geometry>
-                <mesh filename="package://melfa_assista_hardware/meshes/camera_adapter_link.STL" />
+                <mesh filename="file://$(find melfa_assista_hardware)/meshes/camera_adapter_link.STL" />
             </geometry>
             <material name="">
@@ -20,5 +20,5 @@
             <origin xyz="0 0 0" rpy="0 0 0" />
             <geometry>
-                <mesh filename="package://melfa_assista_hardware/meshes/camera_adapter_link.STL" />
+                <mesh filename="file://$(find melfa_assista_hardware)/meshes/camera_adapter_link.STL" />
             </geometry>
         </collision>
@@ -34,5 +34,5 @@
             <origin xyz="0 0 0" rpy="0 0 0" />
             <geometry>
-                <mesh filename="package://melfa_assista_hardware/meshes/camera_link.STL" />
+                <mesh filename="file://$(find melfa_assista_hardware)/meshes/camera_link.STL" />
             </geometry>
             <material name="">
@@ -43,5 +43,5 @@
             <origin xyz="0 0 0" rpy="0 0 0" />
             <geometry>
-                <mesh filename="package://melfa_assista_hardware/meshes/camera_link.STL" />
+                <mesh filename="file://$(find melfa_assista_hardware)/meshes/camera_link.STL" />
             </geometry>
         </collision>
@@ -54,5 +54,5 @@
     </joint>
     <joint name="joint_camera" type="fixed">
-        <origin xyz="0 0.027 -0.0185" rpy="3.1416 0 3.1416" />
+        <origin xyz="0 0.027 -0.0185" rpy="${pi} 0 ${pi}" />
         <parent link="camera_adapter_link" />
         <child link="camera_link" />
@@ -62,9 +62,9 @@
     </link>
     <joint name="joint_camera_optical_frame" type="fixed">
-        <origin xyz="0 0 0" rpy="${-pi/2} 0 ${-pi/2}"/>
+        <origin xyz="0 0 0.06" rpy="-${pi/2} -${pi/2} 0"/>
         <parent link="camera_link" />
         <child link="camera_link_optical" />
     </joint>
-    <gazebo reference="camera_link">
+    <gazebo reference="camera_link_optical">
         <material>Gazebo/Black</material>
         <sensor name="camera" type="camera">

File: melfa_assista_hardware/description/urdf/ros2_control.xacro (robot description, xacro)
@@ -1,24 +1,23 @@
 <?xml version="1.0"?>
 <robot xmlns:xacro="http://www.ros.org/wiki/xacro">
-  <xacro:macro name="melfa_ros2_control"
-    params="name robot_ip use_sim:=^|false use_fake_hardware:=^|true">
-    <ros2_control name="${name}" type="system">
-      <xacro:if value="$(arg use_sim)">
+    <ros2_control name="Assista_Robot_System" type="system">
+      <xacro:if value="$(arg sim_mode)">
         <hardware>
           <plugin>gazebo_ros2_control/GazeboSystem</plugin>
         </hardware>
       </xacro:if>
-      <xacro:unless value="$(arg use_sim)">
+      <!-- <xacro:if value="$(arg use_mockup)">
         <hardware>
-          <xacro:if value="${use_fake_hardware}">
-            <plugin>fake_components/GenericSystem</plugin>
-            <param name="state_following_offset">0.0</param>
-          </xacro:if>
-          <xacro:unless value="${use_fake_hardware}">
-            <plugin>melfa_assista_hardware/MelfaHW</plugin>
-            <param name="robot_ip">${robot_ip}</param>
-          </xacro:unless>
+          <plugin>fake_components/GenericSystem</plugin>
+          <param name="state_following_offset">0.0</param>
+        </hardware>
+      </xacro:if>
+      <xacro:unless value="$(arg use_mockup)">
+        <hardware>
+          <plugin>melfa_assista_hardware/MelfaHW</plugin>
+          <param name="robot_ip">"$(arg robot_ip)"</param>
         </hardware>
       </xacro:unless>
+      -->
       <joint name="joint_1">
         <param name="initial_value">0.0</param>
@@ -79,4 +78,9 @@
       </gpio>
     </ros2_control>
-  </xacro:macro>
+  <!-- Enable Gazebo Plugins -->
+  <gazebo>
+    <plugin filename="libgazebo_ros2_control.so" name="gazebo_ros2_control">
+      <parameters>$(find melfa_assista_hardware)/config/melfa_controller.yaml</parameters>
+    </plugin>
+  </gazebo>
 </robot>

File: melfa_assista_hardware/description/urdf/tool.xacro (robot description, xacro)
@@ -26,19 +26,19 @@
       <geometry>
         <mesh
-          filename="package://melfa_assista_hardware/meshes/coact_base_link.STL" />
-      </geometry>
-      <material
-        name="">
-        <color
-          rgba="0.79216 0.81961 0.93333 1" />
-      </material>
-    </visual>
-    <collision>
-      <origin
-        xyz="0 0 0"
-        rpy="0 0 0" />
-      <geometry>
-        <mesh
-          filename="package://melfa_assista_hardware/meshes/coact_base_link.STL" />
+          filename="file://$(find melfa_assista_hardware)/meshes/coact_base_link.STL" />
+      </geometry>
+      <material
+        name="">
+        <color
+          rgba="0.79216 0.81961 0.93333 1" />
+      </material>
+    </visual>
+    <collision>
+      <origin
+        xyz="0 0 0"
+        rpy="0 0 0" />
+      <geometry>
+        <mesh
+          filename="file://$(find melfa_assista_hardware)/meshes/coact_base_link.STL" />
       </geometry>
     </collision>
@@ -66,19 +66,19 @@
       <geometry>
         <mesh
-          filename="package://melfa_assista_hardware/meshes/housing_link.STL" />
-      </geometry>
-      <material
-        name="">
-        <color
-          rgba="0.79216 0.81961 0.93333 1" />
-      </material>
-    </visual>
-    <collision>
-      <origin
-        xyz="0 0 0"
-        rpy="0 0 0" />
-      <geometry>
-        <mesh
-          filename="package://melfa_assista_hardware/meshes/housing_link.STL" />
+          filename="file://$(find melfa_assista_hardware)/meshes/housing_link.STL" />
+      </geometry>
+      <material
+        name="">
+        <color
+          rgba="0.79216 0.81961 0.93333 1" />
+      </material>
+    </visual>
+    <collision>
+      <origin
+        xyz="0 0 0"
+        rpy="0 0 0" />
+      <geometry>
+        <mesh
+          filename="file://$(find melfa_assista_hardware)/meshes/housing_link.STL" />
       </geometry>
     </collision>
@@ -119,19 +119,19 @@
       <geometry>
         <mesh
-          filename="package://melfa_assista_hardware/meshes/hand_left_link.STL" />
-      </geometry>
-      <material
-        name="">
-        <color
-          rgba="0.79216 0.81961 0.93333 1" />
-      </material>
-    </visual>
-    <collision>
-      <origin
-        xyz="0 0 0"
-        rpy="0 0 0" />
-      <geometry>
-        <mesh
-          filename="package://melfa_assista_hardware/meshes/hand_left_link.STL" />
+          filename="file://$(find melfa_assista_hardware)/meshes/hand_left_link.STL" />
+      </geometry>
+      <material
+        name="">
+        <color
+          rgba="0.79216 0.81961 0.93333 1" />
+      </material>
+    </visual>
+    <collision>
+      <origin
+        xyz="0 0 0"
+        rpy="0 0 0" />
+      <geometry>
+        <mesh
+          filename="file://$(find melfa_assista_hardware)/meshes/hand_left_link.STL" />
       </geometry>
     </collision>
@@ -177,5 +177,5 @@
       <geometry>
         <mesh
-          filename="package://melfa_assista_hardware/meshes/finger_left_link.STL" />
+          filename="file://$(find melfa_assista_hardware)/meshes/finger_left_link.STL" />
       </geometry>
       <material
@@ -191,5 +191,5 @@
       <geometry>
         <mesh
-          filename="package://melfa_assista_hardware/meshes/finger_left_link.STL" />
+          filename="file://$(find melfa_assista_hardware)/meshes/finger_left_link.STL" />
       </geometry>
     </collision>
@@ -230,19 +230,19 @@
       <geometry>
         <mesh
-          filename="package://melfa_assista_hardware/meshes/hand_right_link.STL" />
-      </geometry>
-      <material
-        name="">
-        <color
-          rgba="0.79216 0.81961 0.93333 1" />
-      </material>
-    </visual>
-    <collision>
-      <origin
-        xyz="0 0 0"
-        rpy="0 0 0" />
-      <geometry>
-        <mesh
-          filename="package://melfa_assista_hardware/meshes/hand_right_link.STL" />
+          filename="file://$(find melfa_assista_hardware)/meshes/hand_right_link.STL" />
+      </geometry>
+      <material
+        name="">
+        <color
+          rgba="0.79216 0.81961 0.93333 1" />
+      </material>
+    </visual>
+    <collision>
+      <origin
+        xyz="0 0 0"
+        rpy="0 0 0" />
+      <geometry>
+        <mesh
+          filename="file://$(find melfa_assista_hardware)/meshes/hand_right_link.STL" />
       </geometry>
     </collision>
@@ -267,5 +267,5 @@
     <mimic
       joint="joint_hand_left"
-      multiplier="-1"
+      multiplier="1"
       offset="0" />
   </joint>
@@ -292,19 +292,19 @@
       <geometry>
         <mesh
-          filename="package://melfa_assista_hardware/meshes/finger_right_link.STL" />
-      </geometry>
-      <material
-        name="">
-        <color
-          rgba="0.79216 0.81961 0.93333 1" />
-      </material>
-    </visual>
-    <collision>
-      <origin
-        xyz="0 0 0"
-        rpy="0 0 0" />
-      <geometry>
-        <mesh
-          filename="package://melfa_assista_hardware/meshes/finger_right_link.STL" />
+          filename="file://$(find melfa_assista_hardware)/meshes/finger_right_link.STL" />
+      </geometry>
+      <material
+        name="">
+        <color
+          rgba="0.79216 0.81961 0.93333 1" />
+      </material>
+    </visual>
+    <collision>
+      <origin
+        xyz="0 0 0"
+        rpy="0 0 0" />
+      <geometry>
+        <mesh
+          filename="file://$(find melfa_assista_hardware)/meshes/finger_right_link.STL" />
       </geometry>
     </collision>
@@ -323,3 +323,9 @@
       xyz="0 0 0" />
   </joint>
+  <!-- Tool Joint Connection to the Robot -->
+  <joint name="joint_tool_robot" type="fixed">
+    <origin xyz="0.0 0.0 0.01" rpy="-${(pi/2)} 0.0 ${(pi/2)}"/>
+    <parent link="Link_6_1"/>
+    <child link="coact_base_link"/>
+  </joint>
 </robot>

Commit message: Fixed Issue in Gazebo

File: melfa_assista_hardware/description/urdf/assista_robot.xacro (robot description, xacro)
@@ -145,5 +145,5 @@
 </link>
 <joint name="joint_0" type="fixed">
-  <origin xyz="0 0 0" rpy="0 0 0"/>
+  <origin xyz="0 0 0.001" rpy="0 0 0"/>
   <parent link="world"/>
   <child link="base_link"/>
