Commit message: Renamed STL Files, fixed the real robott launch file

File: melfa_assista_hardware/description/urdf/assista_robot.xacro (robot description, xacro)
@@ -12,5 +12,5 @@
     <origin xyz="0 0 0" rpy="0 0 0"/>
     <geometry>
-      <mesh filename="file://$(find melfa_assista_hardware)/meshes/base_link.STL" scale="0.001 0.001 0.001"/>
+      <mesh filename="file://$(find melfa_assista_hardware)/meshes/base_link.stl" scale="0.001 0.001 0.001"/>
       <cylinder radius="0.5" length="1.0"/>
     </geometry>
@@ -20,5 +20,5 @@
     <origin xyz="0 0 0" rpy="0 0 0"/>
     <geometry>
-      <mesh filename="file://$(find melfa_assista_hardware)/meshes/base_link.STL" scale="0.001 0.001 0.001"/>
+      <mesh filename="file://$(find melfa_assista_hardware)/meshes/base_link.stl" scale="0.001 0.001 0.001"/>
     </geometry>
   </collision>

File: melfa_assista_hardware/description/urdf/camera.xacro (robot description, xacro)
@@ -11,5 +11,5 @@
             <origin xyz="0 0 0" rpy="0 0 0" />
             <geometry>
-                <mesh filename="file://$(find melfa_assista_hardware)/meshes/camera_adapter_link.STL" />
+                <mesh filename="file://$(find melfa_assista_hardware)/meshes/camera_adapter_link.stl" />
             </geometry>
             <material name="">
@@ -20,5 +20,5 @@
             <origin xyz="0 0 0" rpy="0 0 0" />
             <geometry>
-                <mesh filename="file://$(find melfa_assista_hardware)/meshes/camera_adapter_link.STL" />
+                <mesh filename="file://$(find melfa_assista_hardware)/meshes/camera_adapter_link.stl" />
             </geometry>
         </collision>
@@ -34,5 +34,5 @@
             <origin xyz="0 0 0" rpy="0 0 0" />
             <geometry>
-                <mesh filename="file://$(find melfa_assista_hardware)/meshes/camera_link.STL" />
+                <mesh filename="file://$(find melfa_assista_hardware)/meshes/camera_link.stl" />
             </geometry>
             <material name="">
@@ -43,5 +43,5 @@
             <origin xyz="0 0 0" rpy="0 0 0" />
             <geometry>
-                <mesh filename="file://$(find melfa_assista_hardware)/meshes/camera_link.STL" />
+                <mesh filename="file://$(find melfa_assista_hardware)/meshes/camera_link.stl" />
             </geometry>
         </collision>

File: melfa_assista_hardware/description/urdf/ros2_control.xacro (robot description, xacro)
@@ -7,5 +7,5 @@
         </hardware>
       </xacro:if>
-      <!-- <xacro:if value="$(arg use_mockup)">
+      <xacro:if value="$(arg use_mockup)">
         <hardware>
           <plugin>fake_components/GenericSystem</plugin>
@@ -19,5 +19,4 @@
         </hardware>
       </xacro:unless>
-      -->
       <joint name="joint_1">
         <param name="initial_value">0.0</param>

File: melfa_assista_hardware/description/urdf/tool.xacro (robot description, xacro)
@@ -26,19 +26,19 @@
       <geometry>
         <mesh
-          filename="file://$(find melfa_assista_hardware)/meshes/coact_base_link.STL" />
-      </geometry>
-      <material
-        name="">
-        <color
-          rgba="0.79216 0.81961 0.93333 1" />
-      </material>
-    </visual>
-    <collision>
-      <origin
-        xyz="0 0 0"
-        rpy="0 0 0" />
-      <geometry>
-        <mesh
-          filename="file://$(find melfa_assista_hardware)/meshes/coact_base_link.STL" />
+          filename="file://$(find melfa_assista_hardware)/meshes/coact_base_link.stl" />
+      </geometry>
+      <material
+        name="">
+        <color
+          rgba="0.79216 0.81961 0.93333 1" />
+      </material>
+    </visual>
+    <collision>
+      <origin
+        xyz="0 0 0"
+        rpy="0 0 0" />
+      <geometry>
+        <mesh
+          filename="file://$(find melfa_assista_hardware)/meshes/coact_base_link.stl" />
       </geometry>
     </collision>
@@ -66,19 +66,19 @@
       <geometry>
         <mesh
-          filename="file://$(find melfa_assista_hardware)/meshes/housing_link.STL" />
-      </geometry>
-      <material
-        name="">
-        <color
-          rgba="0.79216 0.81961 0.93333 1" />
-      </material>
-    </visual>
-    <collision>
-      <origin
-        xyz="0 0 0"
-        rpy="0 0 0" />
-      <geometry>
-        <mesh
-          filename="file://$(find melfa_assista_hardware)/meshes/housing_link.STL" />
+          filename="file://$(find melfa_assista_hardware)/meshes/housing_link.stl" />
+      </geometry>
+      <material
+        name="">
+        <color
+          rgba="0.79216 0.81961 0.93333 1" />
+      </material>
+    </visual>
+    <collision>
+      <origin
+        xyz="0 0 0"
+        rpy="0 0 0" />
+      <geometry>
+        <mesh
+          filename="file://$(find melfa_assista_hardware)/meshes/housing_link.stl" />
       </geometry>
     </collision>
@@ -119,19 +119,19 @@
       <geometry>
         <mesh
-          filename="file://$(find melfa_assista_hardware)/meshes/hand_left_link.STL" />
-      </geometry>
-      <material
-        name="">
-        <color
-          rgba="0.79216 0.81961 0.93333 1" />
-      </material>
-    </visual>
-    <collision>
-      <origin
-        xyz="0 0 0"
-        rpy="0 0 0" />
-      <geometry>
-        <mesh
-          filename="file://$(find melfa_assista_hardware)/meshes/hand_left_link.STL" />
+          filename="file://$(find melfa_assista_hardware)/meshes/hand_left_link.stl" />
+      </geometry>
+      <material
+        name="">
+        <color
+          rgba="0.79216 0.81961 0.93333 1" />
+      </material>
+    </visual>
+    <collision>
+      <origin
+        xyz="0 0 0"
+        rpy="0 0 0" />
+      <geometry>
+        <mesh
+          filename="file://$(find melfa_assista_hardware)/meshes/hand_left_link.stl" />
       </geometry>
     </collision>
@@ -177,5 +177,5 @@
       <geometry>
         <mesh
-          filename="file://$(find melfa_assista_hardware)/meshes/finger_left_link.STL" />
+          filename="file://$(find melfa_assista_hardware)/meshes/finger_left_link.stl" />
       </geometry>
       <material
@@ -191,5 +191,5 @@
       <geometry>
         <mesh
-          filename="file://$(find melfa_assista_hardware)/meshes/finger_left_link.STL" />
+          filename="file://$(find melfa_assista_hardware)/meshes/finger_left_link.stl" />
       </geometry>
     </collision>
@@ -230,19 +230,19 @@
       <geometry>
         <mesh
-          filename="file://$(find melfa_assista_hardware)/meshes/hand_right_link.STL" />
-      </geometry>
-      <material
-        name="">
-        <color
-          rgba="0.79216 0.81961 0.93333 1" />
-      </material>
-    </visual>
-    <collision>
-      <origin
-        xyz="0 0 0"
-        rpy="0 0 0" />
-      <geometry>
-        <mesh
-          filename="file://$(find melfa_assista_hardware)/meshes/hand_right_link.STL" />
+          filename="file://$(find melfa_assista_hardware)/meshes/hand_right_link.stl" />
+      </geometry>
+      <material
+        name="">
+        <color
+          rgba="0.79216 0.81961 0.93333 1" />
+      </material>
+    </visual>
+    <collision>
+      <origin
+        xyz="0 0 0"
+        rpy="0 0 0" />
+      <geometry>
+        <mesh
+          filename="file://$(find melfa_assista_hardware)/meshes/hand_right_link.stl" />
       </geometry>
     </collision>
@@ -292,19 +292,19 @@
       <geometry>
         <mesh
-          filename="file://$(find melfa_assista_hardware)/meshes/finger_right_link.STL" />
-      </geometry>
-      <material
-        name="">
-        <color
-          rgba="0.79216 0.81961 0.93333 1" />
-      </material>
-    </visual>
-    <collision>
-      <origin
-        xyz="0 0 0"
-        rpy="0 0 0" />
-      <geometry>
-        <mesh
-          filename="file://$(find melfa_assista_hardware)/meshes/finger_right_link.STL" />
+          filename="file://$(find melfa_assista_hardware)/meshes/finger_right_link.stl" />
+      </geometry>
+      <material
+        name="">
+        <color
+          rgba="0.79216 0.81961 0.93333 1" />
+      </material>
+    </visual>
+    <collision>
+      <origin
+        xyz="0 0 0"
+        rpy="0 0 0" />
+      <geometry>
+        <mesh
+          filename="file://$(find melfa_assista_hardware)/meshes/finger_right_link.stl" />
       </geometry>
     </collision>
