Commit message: Added a Gripper Controller to move the Tool

File: melfa_assista_hardware/description/urdf/ros2_control.xacro (robot description, xacro)
@@ -7,15 +7,17 @@
         </hardware>
       </xacro:if>
-      <xacro:if value="$(arg use_mockup)">
-        <hardware>
-          <plugin>fake_components/GenericSystem</plugin>
-          <param name="state_following_offset">0.0</param>
-        </hardware>
-      </xacro:if>
-      <xacro:unless value="$(arg use_mockup)">
-        <hardware>
-          <plugin>melfa_assista_hardware/MelfaHW</plugin>
-          <param name="robot_ip">"$(arg robot_ip)"</param>
-        </hardware>
+      <xacro:unless value="$(arg sim_mode)">
+        <xacro:if value="$(arg use_mockup)">
+          <hardware>
+            <plugin>fake_components/GenericSystem</plugin>
+            <param name="state_following_offset">0.0</param>
+          </hardware>
+        </xacro:if>
+        <xacro:unless value="$(arg use_mockup)">
+          <hardware>
+            <plugin>melfa_assista_hardware/MelfaHW</plugin>
+            <param name="robot_ip">"$(arg robot_ip)"</param>
+          </hardware>
+        </xacro:unless>
       </xacro:unless>
       <joint name="joint_1">
@@ -67,4 +69,13 @@
         <state_interface name="position" />
       </joint>
+      <joint name="joint_hand_left">
+        <param name="initial_value">0.0</param>
+        <command_interface name="position">
+          <param name="min">0</param>
+          <param name="max">0.006</param>
+        </command_interface>
+        <state_interface name="position" />
+        <state_interface name="velocity"/>
+      </joint>
       <!-- from https://github.com/ros-controls/ros2_control/blob/f58d4072dbd1c3fd4e1f64cd10a19a2b60f59049/ros2_control_test_assets/include/ros2_control_test_assets/components_urdfs.hpp#L344 -->
       <gpio name="tool_flansch">

Commit message: Added the Gripper Action Controller to the Interface

File: melfa_assista_hardware/description/urdf/ros2_control.xacro (robot description, xacro)
@@ -89,8 +89,10 @@
     </ros2_control>
   <!-- Enable Gazebo Plugins -->
-  <gazebo>
-    <plugin filename="libgazebo_ros2_control.so" name="gazebo_ros2_control">
-      <parameters>$(find melfa_assista_hardware)/config/melfa_controller.yaml</parameters>
-    </plugin>
-  </gazebo>
+  <xacro:if value="$(arg sim_mode)">
+    <gazebo>
+      <plugin filename="libgazebo_ros2_control.so" name="gazebo_ros2_control">
+        <parameters>$(find melfa_assista_hardware)/config/melfa_controller.yaml</parameters>
+      </plugin>
+    </gazebo>
+  </xacro:if>
 </robot>

File: melfa_assista_hardware/description/urdf/tool.xacro (robot description, xacro)
@@ -137,7 +137,5 @@
     </collision>
   </link>
-  <joint
-    name="joint_hand_left"
-    type="prismatic">
+  <joint name="joint_hand_left" type="prismatic">
     <origin
       xyz="0 0 0.0122"

Commit message: Finger now are Moving

File: melfa_assista_hardware/description/urdf/ros2_control.xacro (robot description, xacro)
@@ -78,4 +78,12 @@
         <state_interface name="velocity"/>
       </joint>
+      <joint name="joint_hand_right">
+        <param name="mimic">joint_hand_left</param>
+        <param name="multiplier">1</param>
+        <command_interface name="position"/>
+        <state_interface name="position"/>
+        <state_interface name="velocity"/>
+        <state_interface name="effort"/>
+      </joint>
       <!-- from https://github.com/ros-controls/ros2_control/blob/f58d4072dbd1c3fd4e1f64cd10a19a2b60f59049/ros2_control_test_assets/include/ros2_control_test_assets/components_urdfs.hpp#L344 -->
       <gpio name="tool_flansch">

File: melfa_assista_hardware/description/urdf/tool.xacro (robot description, xacro)
@@ -1,7 +1,8 @@
 <?xml version="1.0" encoding="utf-8"?>
-<!-- This URDF was automatically created by SolidWorks to URDF Exporter! Originally created by Stephen Brawner (brawner@gmail.com)
+<!-- This URDF was automatically created by SolidWorks to URDF Exporter! Originally created by
+Stephen Brawner (brawner@gmail.com)
      Commit Version: 1.6.0-4-g7f85cfe  Build Version: 1.6.7995.38578
      For more information, please see http://wiki.ros.org/sw_urdf_exporter -->
-  <robot xmlns:xacro="http://www.ros.org/wiki/xacro">
+<robot xmlns:xacro="http://www.ros.org/wiki/xacro">
   <link
     name="coact_base_link">
@@ -247,5 +248,5 @@
   </link>
   <joint
-    name="hand_right_joint"
+    name="joint_hand_right"
     type="prismatic">
     <origin
@@ -263,8 +264,5 @@
       effort="200"
       velocity="1.0" />
-    <mimic
-      joint="joint_hand_left"
-      multiplier="-1"
-      offset="0" />
+    <mimic joint="joint_hand_left" />
   </joint>
   <link
@@ -323,7 +321,7 @@
   <!-- Tool Joint Connection to the Robot -->
   <joint name="joint_tool_robot" type="fixed">
-    <origin xyz="0.0 0.0 0.01" rpy="-${(pi/2)} 0.0 ${(pi/2)}"/>
-    <parent link="Link_6_1"/>
-    <child link="coact_base_link"/>
+    <origin xyz="0.0 0.0 0.01" rpy="-${(pi/2)} 0.0 ${(pi/2)}" />
+    <parent link="Link_6_1" />
+    <child link="coact_base_link" />
   </joint>
 </robot>
