Commit message: Added the sensopart Camera and TCPs to the Interface

File: melfa_assista_hardware/description/urdf/camera.xacro (robot description, xacro)
@@ -1,69 +1,117 @@
 <?xml version="1.0" encoding="utf-8"?>
 <robot xmlns:xacro="http://www.ros.org/wiki/xacro">
-    <link name="camera_adapter_link">
-        <inertial>
-            <origin xyz="6.8987E-05 6.8987E-05 0.0086472" rpy="0 0 0" />
-            <mass value="0.11061" />
-            <inertia ixx="0.00011703" ixy="-7.4547E-10" ixz="3.2264E-07" iyy="0.00012118"
-                iyz="-6.0814E-08" izz="2.26E-05" />
-        </inertial>
-        <visual>
-            <origin xyz="0 0 0" rpy="0 0 0" />
-            <geometry>
-                <mesh filename="file://$(find melfa_assista_hardware)/meshes/camera_adapter_link.stl" />
-            </geometry>
-            <material name="">
-                <color rgba="1 1 1 1" />
-            </material>
-        </visual>
-        <collision>
-            <origin xyz="0 0 0" rpy="0 0 0" />
-            <geometry>
-                <mesh filename="file://$(find melfa_assista_hardware)/meshes/camera_adapter_link.stl" />
-            </geometry>
-        </collision>
-    </link>
-    <link name="camera_link">
-        <inertial>
-            <origin xyz="6.8987E-05 8.2543E-06 0.0086472" rpy="0 0 0" />
-            <mass value="0.11061" />
-            <inertia ixx="0.00011703" ixy="-7.4547E-10" ixz="3.2264E-07" iyy="0.00012118"
-                iyz="-6.0814E-08" izz="2.26E-05" />
-        </inertial>
-        <visual>
-            <origin xyz="0 0 0" rpy="0 0 0" />
-            <geometry>
-                <mesh filename="file://$(find melfa_assista_hardware)/meshes/camera_link.stl" />
-            </geometry>
-            <material name="">
-                <color rgba="0.50196 0.50196 0.50196 1" />
-            </material>
-        </visual>
-        <collision>
-            <origin xyz="0 0 0" rpy="0 0 0" />
-            <geometry>
-                <mesh filename="file://$(find melfa_assista_hardware)/meshes/camera_link.stl" />
-            </geometry>
-        </collision>
-    </link>
-    <joint name="joint_camera_adapter" type="fixed">
-        <origin xyz="-0.00275 -0.0425 -0.04425" rpy="-1.5708 0 0" />
-        <parent link="coact_base_link" />
-        <child link="camera_adapter_link" />
-        <axis xyz="0 0 0" />
-    </joint>
-    <joint name="joint_camera" type="fixed">
-        <origin xyz="0 0.027 -0.0185" rpy="${pi} 0 ${pi}" />
-        <parent link="camera_adapter_link" />
-        <child link="camera_link" />
-        <axis xyz="0 0 0" />
-    </joint>
-    <link name="camera_link_optical">
-    </link>
-    <joint name="joint_camera_optical_frame" type="fixed">
-        <origin xyz="0 0 0.06" rpy="-${pi/2} -${pi/2} 0"/>
-        <parent link="camera_link" />
-        <child link="camera_link_optical" />
-    </joint>
+  <link
+  name="camera_adapter_link">
+  <inertial>
+    <origin
+      xyz="-0.026 -0.022971 -1.0408E-17"
+      rpy="0 0 0" />
+    <mass
+      value="0.16292" />
+    <inertia
+      ixx="6.5111E-05"
+      ixy="-2.7068E-05"
+      ixz="-5.9292E-21"
+      iyy="3.0709E-05"
+      iyz="-9.3174E-21"
+      izz="7.4701E-05" />
+  </inertial>
+  <visual>
+    <origin
+      xyz="0 0 0"
+      rpy="0 0 0" />
+    <geometry>
+      <mesh
+        filename="file://$(find melfa_assista_hardware)/meshes/camera_adapter_link.stl" />
+    </geometry>
+    <material
+      name="">
+      <color
+        rgba="0.64706 0.61961 0.58824 1" />
+    </material>
+  </visual>
+  <collision>
+    <origin
+      xyz="0 0 0"
+      rpy="0 0 0" />
+    <geometry>
+      <mesh
+        filename="file://$(find melfa_assista_hardware)/meshes/camera_adapter_link.stl" />
+    </geometry>
+  </collision>
+</link>
+<joint
+  name="camera_adapter_joint"
+  type="fixed">
+  <origin
+    xyz="0.033234 0.033234 -0.0041"
+    rpy="-1.5708 0 -2.3562" />
+  <parent
+    link="coact_base_link" />
+  <child
+    link="camera_adapter_link" />
+  <axis
+    xyz="0 0 0" />
+</joint>
+<link
+  name="camera_link">
+  <inertial>
+    <origin
+      xyz="-6.8696E-07 -0.00043025 0.03599"
+      rpy="0 0 0" />
+    <mass
+      value="0.13788" />
+    <inertia
+      ixx="8.1425E-05"
+      ixy="-1.5749E-10"
+      ixz="1.2373E-08"
+      iyy="8.2407E-05"
+      iyz="9.6107E-07"
+      izz="4.3666E-05" />
+  </inertial>
+  <visual>
+    <origin
+      xyz="0 0 0"
+      rpy="0 ${(pi)} ${(pi)}" />
+    <geometry>
+      <mesh
+        filename="file://$(find melfa_assista_hardware)/meshes/camera_link.stl" />
+    </geometry>
+    <material
+      name="">
+      <color
+        rgba="0.74902 0.74902 0.74902 1" />
+    </material>
+  </visual>
+  <collision>
+    <origin
+      xyz="0 0 0"
+      rpy="0 0 0" />
+    <geometry>
+      <mesh
+        filename="file://$(find melfa_assista_hardware)/meshes/camera_link.stl" />
+    </geometry>
+  </collision>
+</link>
+<joint
+  name="camera_joint"
+  type="fixed">
+  <origin
+    xyz="-0.067443 -0.054897 0"
+    rpy="${-(1.3937) + pi} 1.5708 0" />
+  <parent
+    link="camera_adapter_link" />
+  <child
+    link="camera_link" />
+  <axis
+    xyz="0 0 0" />
+</joint>
+<link name="camera_tcp">
+</link>
+<joint name="camera_tcp_joint" type="fixed">
+  <origin xyz="0.0 0.0 0.0" rpy="0.0 0.0 0.0"/>
+  <parent link="camera_link"/>
+  <child link="camera_tcp"/>
+</joint>
     <gazebo reference="camera_link_optical">
         <material>Gazebo/Black</material>

File: melfa_assista_hardware/description/urdf/ros2_control.xacro (robot description, xacro)
@@ -84,5 +84,4 @@
         <state_interface name="position"/>
         <state_interface name="velocity"/>
-        <state_interface name="effort"/>
       </joint>
       <!-- from https://github.com/ros-controls/ros2_control/blob/f58d4072dbd1c3fd4e1f64cd10a19a2b60f59049/ros2_control_test_assets/include/ros2_control_test_assets/components_urdfs.hpp#L344 -->

File: melfa_assista_hardware/description/urdf/tool.xacro (robot description, xacro)
@@ -1,22 +1,21 @@
 <?xml version="1.0" encoding="utf-8"?>
-<!-- This URDF was automatically created by SolidWorks to URDF Exporter! Originally created by
-Stephen Brawner (brawner@gmail.com)
+<!-- This URDF was automatically created by SolidWorks to URDF Exporter! Originally created by Stephen Brawner (brawner@gmail.com)
      Commit Version: 1.6.0-4-g7f85cfe  Build Version: 1.6.7995.38578
      For more information, please see http://wiki.ros.org/sw_urdf_exporter -->
-<robot xmlns:xacro="http://www.ros.org/wiki/xacro">
+<robot>
   <link
     name="coact_base_link">
     <inertial>
       <origin
-        xyz="-0.0035845 0.0019636 0.012011"
+        xyz="0.0011461 -3.4094E-05 -0.011589"
         rpy="0 0 0" />
       <mass
         value="0.07902" />
       <inertia
-        ixx="4.1882E-05"
-        ixy="2.5898E-07"
-        ixz="-4.4967E-07"
-        iyy="3.7898E-05"
-        iyz="-3.1583E-07"
+        ixx="4.0149E-05"
+        ixy="-1.9916E-06"
+        ixz="5.4129E-07"
+        iyy="3.9631E-05"
+        iyz="-9.4644E-08"
         izz="7.2725E-05" />
     </inertial>
@@ -45,9 +44,22 @@
     </collision>
   </link>
+  <joint
+    name="coact_base_joint"
+    type="fixed">
+    <origin
+      xyz="0 0 0.0321"
+      rpy="0 0 -${(45 * (pi/180))}" />
+    <parent
+      link="Link_6_1" />
+    <child
+      link="coact_base_link" />
+    <axis
+      xyz="0 0 0" />
+  </joint>
   <link
     name="housing_link">
     <inertial>
       <origin
-        xyz="0.0004679 -7.9733E-06 -0.071807"
+        xyz="0.0004679 -7.9786E-06 -0.071807"
         rpy="0 0 0" />
       <mass
@@ -55,9 +67,9 @@
       <inertia
         ixx="0.00050627"
-        ixy="5.502E-08"
-        ixz="-1.027E-07"
+        ixy="5.4844E-08"
+        ixz="-1.0292E-07"
         iyy="0.00055192"
-        iyz="4.1906E-08"
-        izz="0.00032568" />
+        iyz="4.2618E-08"
+        izz="0.00032569" />
     </inertial>
     <visual>
@@ -89,6 +101,6 @@
     type="fixed">
     <origin
-      xyz="-0.00274999999999998 -0.1325 0.00274999999999998"
-      rpy="1.5707963267949 0 0" />
+      xyz="0 0 0.1089"
+      rpy="0 0 2.3562" />
     <parent
       link="coact_base_link" />
@@ -102,5 +114,5 @@
     <inertial>
       <origin
-        xyz="0.0015172 -0.015033 0.0033678"
+        xyz="-0.00091365 -0.015033 0.0033678"
         rpy="0 0 0" />
       <mass
@@ -138,8 +150,10 @@
     </collision>
   </link>
-  <joint name="joint_hand_left" type="prismatic">
+  <joint
+    name="joint_hand_left"
+    type="prismatic">
     <origin
       xyz="0 0 0.0122"
-      rpy="1.5708 0 0" />
+      rpy="1.5708 0 3.1416" />
     <parent
       link="housing_link" />
@@ -149,8 +163,8 @@
       xyz="1 0 0" />
     <limit
-      lower="0.0"
-      upper="0.006"
-      effort="200"
-      velocity="1.0" />
+      lower="0"
+      upper="0.03"
+      effort="120"
+      velocity="0.5" />
   </joint>
   <link
@@ -158,15 +172,15 @@
     <inertial>
       <origin
-        xyz="0.01141 1.352E-08 0.024079"
-        rpy="0 0 0" />
-      <mass
-        value="0.013672" />
-      <inertia
-        ixx="2.7756E-06"
-        ixy="-5.3984E-13"
-        ixz="1.3676E-07"
-        iyy="2.5808E-06"
-        iyz="1.4625E-12"
-        izz="7.7774E-07" />
+        xyz="0.01141 1.453E-08 0.024079"
+        rpy="0 0 0" />
+      <mass
+        value="0.011888" />
+      <inertia
+        ixx="2.4136E-06"
+        ixy="-7.1143E-13"
+        ixz="1.1892E-07"
+        iyy="2.2441E-06"
+        iyz="1.2315E-12"
+        izz="6.7629E-07" />
     </inertial>
     <visual>
@@ -181,5 +195,5 @@
         name="">
         <color
-          rgba="0.79608 0.82353 0.93725 1" />
+          rgba="0.79216 0.81961 0.93333 1" />
       </material>
     </visual>
@@ -198,5 +212,5 @@
     type="fixed">
     <origin
-      xyz="0.0080313 -0.012 0"
+      xyz="0.0056005 -0.012 0"
       rpy="-1.5708 0 0" />
     <parent
@@ -211,5 +225,5 @@
     <inertial>
       <origin
-        xyz="0.0015161 -0.015033 0.0033678"
+        xyz="-0.0011169 -0.015033 0.0033678"
         rpy="0 0 0" />
       <mass
@@ -252,5 +266,5 @@
     <origin
       xyz="0 0 0.0122"
-      rpy="1.5708 0 -3.1416" />
+      rpy="1.5708 0 0" />
     <parent
       link="housing_link" />
@@ -260,47 +274,50 @@
       xyz="1 0 0" />
     <limit
-      lower="0.0"
-      upper="0.006"
-      effort="200"
-      velocity="1.0" />
-    <mimic joint="joint_hand_left" />
-  </joint>
-  <link
-    name="finger_right_link">
-    <inertial>
-      <origin
-        xyz="0.01141 1.352E-08 0.024079"
-        rpy="0 0 0" />
-      <mass
-        value="0.011888" />
-      <inertia
-        ixx="2.4136E-06"
-        ixy="-4.6943E-13"
-        ixz="1.1892E-07"
-        iyy="2.2441E-06"
-        iyz="1.2718E-12"
-        izz="6.7629E-07" />
-    </inertial>
-    <visual>
-      <origin
-        xyz="0 0 0"
-        rpy="0 0 0" />
-      <geometry>
-        <mesh
-          filename="file://$(find melfa_assista_hardware)/meshes/finger_right_link.stl" />
-      </geometry>
-      <material
-        name="">
-        <color
-          rgba="0.79216 0.81961 0.93333 1" />
-      </material>
-    </visual>
-    <collision>
-      <origin
-        xyz="0 0 0"
-        rpy="0 0 0" />
-      <geometry>
-        <mesh
-          filename="file://$(find melfa_assista_hardware)/meshes/finger_right_link.stl" />
+      lower="0"
+      upper="0.03"
+      effort="120"
+      velocity="0.5" />
+    <mimic
+      joint="joint_hand_left"
+      multiplier="1"
+      offset="0" />
+  </joint>
+  <link
+    name="finger_right_joint">
+    <inertial>
+      <origin
+        xyz="0.01141 1.453E-08 0.024079"
+        rpy="0 0 0" />
+      <mass
+        value="0.013672" />
+      <inertia
+        ixx="2.7756E-06"
+        ixy="-8.1815E-13"
+        ixz="1.3676E-07"
+        iyy="2.5808E-06"
+        iyz="1.4163E-12"
+        izz="7.7774E-07" />
+    </inertial>
+    <visual>
+      <origin
+        xyz="0 0 0"
+        rpy="0 0 0" />
+      <geometry>
+        <mesh
+          filename="file://$(find melfa_assista_hardware)/meshes/finger_right_joint.stl" />
+      </geometry>
+      <material
+        name="">
+        <color
+          rgba="0.79608 0.82353 0.93725 1" />
+      </material>
+    </visual>
+    <collision>
+      <origin
+        xyz="0 0 0"
+        rpy="0 0 0" />
+      <geometry>
+        <mesh
+          filename="file://$(find melfa_assista_hardware)/meshes/finger_right_joint.stl" />
       </geometry>
     </collision>
@@ -310,18 +327,19 @@
     type="fixed">
     <origin
-      xyz="0.0080302 -0.012 0"
+      xyz="0.0053973 -0.012 0"
       rpy="-1.5708 0 0" />
     <parent
       link="hand_right_link" />
     <child
-      link="finger_right_link" />
+      link="finger_right_joint" />
     <axis
       xyz="0 0 0" />
   </joint>
-  <!-- Tool Joint Connection to the Robot -->
-  <joint name="joint_tool_robot" type="fixed">
-    <origin xyz="0.0 0.0 0.01" rpy="-${(pi/2)} 0.0 ${(pi/2)}" />
-    <parent link="Link_6_1" />
-    <child link="coact_base_link" />
+  <link name="tcp_gripper">
+  </link>
+  <joint name="tcp_joint" type="fixed">
+    <origin xyz="0.0 0.0 0.182" rpy="0.0 0.0 0.0"/>
+    <parent link="Link_6_1"/>
+    <child link="tcp_gripper"/>
   </joint>
 </robot>

Commit message: Fixed the Rotation of the Camera TCP to the World
rotate -90 deg around z

File: melfa_assista_hardware/description/urdf/camera.xacro (robot description, xacro)
@@ -110,5 +110,5 @@
 </link>
 <joint name="camera_tcp_joint" type="fixed">
-  <origin xyz="0.0 0.0 0.0" rpy="0.0 0.0 0.0"/>
+  <origin xyz="0.0 0.0 0.0" rpy="0.0 0.0 -${(90 * pi /180)}"/>
   <parent link="camera_link"/>
   <child link="camera_tcp"/>
