Commit message: Refactor of URDF Files

File: melfa_assista_hardware/description/urdf/camera.xacro (robot description, xacro)
@@ -1,121 +1,70 @@
-<?xml version="1.0" encoding="utf-8"?>
+<?xml version="1.0" encoding="UTF-8"?>
 <robot xmlns:xacro="http://www.ros.org/wiki/xacro">
-  <link
-  name="camera_adapter_link">
-  <inertial>
-    <origin
-      xyz="-0.026 -0.022971 -1.0408E-17"
-      rpy="0 0 0" />
-    <mass
-      value="0.16292" />
-    <inertia
-      ixx="6.5111E-05"
-      ixy="-2.7068E-05"
-      ixz="-5.9292E-21"
-      iyy="3.0709E-05"
-      iyz="-9.3174E-21"
-      izz="7.4701E-05" />
-  </inertial>
-  <visual>
-    <origin
-      xyz="0 0 0"
-      rpy="0 0 0" />
-    <geometry>
-      <mesh
-        filename="file://$(find melfa_assista_hardware)/meshes/camera_adapter_link.stl" />
-    </geometry>
-    <material
-      name="">
-      <color
-        rgba="0.64706 0.61961 0.58824 1" />
-    </material>
-  </visual>
-  <collision>
-    <origin
-      xyz="0 0 0"
-      rpy="0 0 0" />
-    <geometry>
-      <mesh
-        filename="file://$(find melfa_assista_hardware)/meshes/camera_adapter_link.stl" />
-    </geometry>
-  </collision>
-</link>
-<joint
-  name="camera_adapter_joint"
-  type="fixed">
-  <origin
-    xyz="0.033234 0.033234 -0.0041"
-    rpy="-1.5708 0 -2.3562" />
-  <parent
-    link="coact_base_link" />
-  <child
-    link="camera_adapter_link" />
-  <axis
-    xyz="0 0 0" />
-</joint>
-<link
-  name="camera_link">
-  <inertial>
-    <origin
-      xyz="-6.8696E-07 -0.00043025 0.03599"
-      rpy="0 0 0" />
-    <mass
-      value="0.13788" />
-    <inertia
-      ixx="8.1425E-05"
-      ixy="-1.5749E-10"
-      ixz="1.2373E-08"
-      iyy="8.2407E-05"
-      iyz="9.6107E-07"
-      izz="4.3666E-05" />
-  </inertial>
-  <visual>
-    <origin
-      xyz="0 0 0"
-      rpy="0 ${(pi)} ${(pi)}" />
-    <geometry>
-      <mesh
-        filename="file://$(find melfa_assista_hardware)/meshes/camera_link.stl" />
-    </geometry>
-    <material
-      name="">
-      <color
-        rgba="0.74902 0.74902 0.74902 1" />
-    </material>
-  </visual>
-  <collision>
-    <origin
-      xyz="0 0 0"
-      rpy="0 0 0" />
-    <geometry>
-      <mesh
-        filename="file://$(find melfa_assista_hardware)/meshes/camera_link.stl" />
-    </geometry>
-  </collision>
-</link>
-<joint
-  name="camera_joint"
-  type="fixed">
-  <origin
-    xyz="-0.067443 -0.054897 0"
-    rpy="${-(1.3937) + pi} 1.5708 0" />
-  <parent
-    link="camera_adapter_link" />
-  <child
-    link="camera_link" />
-  <axis
-    xyz="0 0 0" />
-</joint>
-<link name="camera_tcp">
-</link>
-<joint name="camera_tcp_joint" type="fixed">
-  <origin xyz="0.0 0.0 0.0" rpy="0.0 0.0 -${(90 * pi /180)}"/>
-  <parent link="camera_link"/>
-  <child link="camera_tcp"/>
-</joint>
+    <link name="camera_adapter_link">
+        <inertial>
+            <origin xyz="-0.026 -0.022971 -1.0408E-17" rpy="0 0 0" />
+            <mass value="0.16292" />
+            <inertia ixx="6.5111E-05" ixy="-2.7068E-05" ixz="-5.9292E-21" iyy="3.0709E-05" iyz="-9.3174E-21" izz="7.4701E-05" />
+        </inertial>
+        <visual>
+            <origin xyz="0 0 0" rpy="0 0 0" />
+            <geometry>
+                <mesh filename="file://$(find melfa_assista_hardware)/meshes/camera_adapter_link.stl" />
+            </geometry>
+            <material name="">
+                <color rgba="0.64706 0.61961 0.58824 1" />
+            </material>
+        </visual>
+        <collision>
+            <origin xyz="0 0 0" rpy="0 0 0" />
+            <geometry>
+                <mesh filename="file://$(find melfa_assista_hardware)/meshes/camera_adapter_link.stl" />
+            </geometry>
+        </collision>
+    </link>
+    <joint name="camera_adapter_joint" type="fixed">
+        <origin xyz="0.033234 0.033234 -0.0041" rpy="-1.5708 0 -2.3562" />
+        <parent link="coact_base_link" />
+        <child link="camera_adapter_link" />
+        <axis xyz="0 0 0" />
+    </joint>
+    <link name="camera_link">
+        <inertial>
+            <origin xyz="-6.8696E-07 -0.00043025 0.03599" rpy="0 0 0" />
+            <mass value="0.13788" />
+            <inertia ixx="8.1425E-05" ixy="-1.5749E-10" ixz="1.2373E-08" iyy="8.2407E-05" iyz="9.6107E-07" izz="4.3666E-05" />
+        </inertial>
+        <visual>
+            <origin xyz="0 0 0" rpy="0 ${(pi)} ${(pi)}" />
+            <geometry>
+                <mesh filename="file://$(find melfa_assista_hardware)/meshes/camera_link.stl" />
+            </geometry>
+            <material name="">
+                <color rgba="0.74902 0.74902 0.74902 1" />
+            </material>
+        </visual>
+        <collision>
+            <origin xyz="0 0 0" rpy="0 ${(pi)} ${(pi)}" />
+            <geometry>
+                <mesh filename="file://$(find melfa_assista_hardware)/meshes/camera_link.stl" />
+            </geometry>
+        </collision>
+    </link>
+    <joint name="camera_joint" type="fixed">
+        <origin xyz="-0.067443 -0.054897 0" rpy="${-(1.3937) + pi} 1.5708 0" />
+        <parent link="camera_adapter_link" />
+        <child link="camera_link" />
+        <axis xyz="0 0 0" />
+    </joint>
+    <link name="camera_tcp" />
+    <joint name="camera_tcp_joint" type="fixed">
+        <origin xyz="0.0 0.0 0.0" rpy="0.0 0.0 -${(90 * pi /180)}" />
+        <parent link="camera_link" />
+        <child link="camera_tcp" />
+    </joint>
     <gazebo reference="camera_link_optical">
         <material>Gazebo/Black</material>
         <sensor name="camera" type="camera">
-            <pose> 0 0 0 0 0 0 </pose>
+            <pose>0 0 0 0 0 0</pose>
             <visualize>true</visualize>
             <update_rate>30</update_rate>

File: melfa_assista_hardware/description/urdf/tool.xacro (robot description, xacro)
@@ -1,345 +1,183 @@
-<?xml version="1.0" encoding="utf-8"?>
+<?xml version="1.0" encoding="UTF-8"?>
 <!-- This URDF was automatically created by SolidWorks to URDF Exporter! Originally created by Stephen Brawner (brawner@gmail.com)
      Commit Version: 1.6.0-4-g7f85cfe  Build Version: 1.6.7995.38578
      For more information, please see http://wiki.ros.org/sw_urdf_exporter -->
 <robot>
-  <link
-    name="coact_base_link">
+  <link name="coact_base_link">
     <inertial>
-      <origin
-        xyz="0.0011461 -3.4094E-05 -0.011589"
-        rpy="0 0 0" />
-      <mass
-        value="0.07902" />
-      <inertia
-        ixx="4.0149E-05"
-        ixy="-1.9916E-06"
-        ixz="5.4129E-07"
-        iyy="3.9631E-05"
-        iyz="-9.4644E-08"
-        izz="7.2725E-05" />
+      <origin xyz="0.0011461 -3.4094E-05 -0.011589" rpy="0 0 0" />
+      <mass value="0.07902" />
+      <inertia ixx="4.0149E-05" ixy="-1.9916E-06" ixz="5.4129E-07" iyy="3.9631E-05" iyz="-9.4644E-08" izz="7.2725E-05" />
     </inertial>
     <visual>
-      <origin
-        xyz="0 0 0"
-        rpy="0 0 0" />
+      <origin xyz="0 0 0" rpy="0 0 0" />
       <geometry>
-        <mesh
-          filename="file://$(find melfa_assista_hardware)/meshes/coact_base_link.stl" />
+        <mesh filename="file://$(find melfa_assista_hardware)/meshes/coact_base_link.stl" />
       </geometry>
-      <material
-        name="">
-        <color
-          rgba="0.79216 0.81961 0.93333 1" />
+      <material name="">
+        <color rgba="0.79216 0.81961 0.93333 1" />
       </material>
     </visual>
     <collision>
-      <origin
-        xyz="0 0 0"
-        rpy="0 0 0" />
+      <origin xyz="0 0 0" rpy="0 0 0" />
       <geometry>
-        <mesh
-          filename="file://$(find melfa_assista_hardware)/meshes/coact_base_link.stl" />
+        <mesh filename="file://$(find melfa_assista_hardware)/meshes/coact_base_link.stl" />
       </geometry>
     </collision>
   </link>
-  <joint
-    name="coact_base_joint"
-    type="fixed">
-    <origin
-      xyz="0 0 0.0321"
-      rpy="0 0 -${(45 * (pi/180))}" />
-    <parent
-      link="Link_6_1" />
-    <child
-      link="coact_base_link" />
-    <axis
-      xyz="0 0 0" />
+  <joint name="coact_base_joint" type="fixed">
+    <origin xyz="0 0 0.0321" rpy="0 0 -${(45 * (pi/180))}" />
+    <parent link="Link_6_1" />
+    <child link="coact_base_link" />
+    <axis xyz="0 0 0" />
   </joint>
-  <link
-    name="housing_link">
+  <link name="housing_link">
     <inertial>
-      <origin
-        xyz="0.0004679 -7.9786E-06 -0.071807"
-        rpy="0 0 0" />
-      <mass
-        value="0.38897" />
-      <inertia
-        ixx="0.00050627"
-        ixy="5.4844E-08"
-        ixz="-1.0292E-07"
-        iyy="0.00055192"
-        iyz="4.2618E-08"
-        izz="0.00032569" />
+      <origin xyz="0.0004679 -7.9786E-06 -0.071807" rpy="0 0 0" />
+      <mass value="0.38897" />
+      <inertia ixx="0.00050627" ixy="5.4844E-08" ixz="-1.0292E-07" iyy="0.00055192" iyz="4.2618E-08" izz="0.00032569" />
     </inertial>
     <visual>
-      <origin
-        xyz="0 0 0"
-        rpy="0 0 0" />
+      <origin xyz="0 0 0" rpy="0 0 0" />
       <geometry>
-        <mesh
-          filename="file://$(find melfa_assista_hardware)/meshes/housing_link.stl" />
+        <mesh filename="file://$(find melfa_assista_hardware)/meshes/housing_link.stl" />
       </geometry>
-      <material
-        name="">
-        <color
-          rgba="0.79216 0.81961 0.93333 1" />
+      <material name="">
+        <color rgba="0.79216 0.81961 0.93333 1" />
       </material>
     </visual>
     <collision>
-      <origin
-        xyz="0 0 0"
-        rpy="0 0 0" />
+      <origin xyz="0 0 0" rpy="0 0 0" />
       <geometry>
-        <mesh
-          filename="file://$(find melfa_assista_hardware)/meshes/housing_link.stl" />
+        <mesh filename="file://$(find melfa_assista_hardware)/meshes/housing_link.stl" />
       </geometry>
     </collision>
   </link>
-  <joint
-    name="housing_joint"
-    type="fixed">
-    <origin
-      xyz="0 0 0.1089"
-      rpy="0 0 2.3562" />
-    <parent
-      link="coact_base_link" />
-    <child
-      link="housing_link" />
-    <axis
-      xyz="0 0 0" />
+  <joint name="housing_joint" type="fixed">
+    <origin xyz="0 0 0.1089" rpy="0 0 2.3562" />
+    <parent link="coact_base_link" />
+    <child link="housing_link" />
+    <axis xyz="0 0 0" />
   </joint>
-  <link
-    name="hand_left_link">
+  <link name="hand_left_link">
     <inertial>
-      <origin
-        xyz="-0.00091365 -0.015033 0.0033678"
-        rpy="0 0 0" />
-      <mass
-        value="0.0034696" />
-      <inertia
-        ixx="2.1052E-07"
-        ixy="-1.1835E-07"
-        ixz="4.2799E-08"
-        iyy="4.0216E-07"
-        iyz="4.2388E-08"
-        izz="5.2415E-07" />
+      <origin xyz="-0.00091365 -0.015033 0.0033678" rpy="0 0 0" />
+      <mass value="0.0034696" />
+      <inertia ixx="2.1052E-07" ixy="-1.1835E-07" ixz="4.2799E-08" iyy="4.0216E-07" iyz="4.2388E-08" izz="5.2415E-07" />
     </inertial>
     <visual>
-      <origin
-        xyz="0 0 0"
-        rpy="0 0 0" />
+      <origin xyz="0 0 0" rpy="0 0 0" />
       <geometry>
-        <mesh
-          filename="file://$(find melfa_assista_hardware)/meshes/hand_left_link.stl" />
+        <mesh filename="file://$(find melfa_assista_hardware)/meshes/hand_left_link.stl" />
       </geometry>
-      <material
-        name="">
-        <color
-          rgba="0.79216 0.81961 0.93333 1" />
+      <material name="">
+        <color rgba="0.79216 0.81961 0.93333 1" />
       </material>
     </visual>
     <collision>
-      <origin
-        xyz="0 0 0"
-        rpy="0 0 0" />
+      <origin xyz="0 0 0" rpy="0 0 0" />
       <geometry>
-        <mesh
-          filename="file://$(find melfa_assista_hardware)/meshes/hand_left_link.stl" />
+        <mesh filename="file://$(find melfa_assista_hardware)/meshes/hand_left_link.stl" />
       </geometry>
     </collision>
   </link>
-  <joint
-    name="joint_hand_left"
-    type="prismatic">
-    <origin
-      xyz="0 0 0.0122"
-      rpy="1.5708 0 3.1416" />
-    <parent
-      link="housing_link" />
-    <child
-      link="hand_left_link" />
-    <axis
-      xyz="1 0 0" />
-    <limit
-      lower="0"
-      upper="0.03"
-      effort="120"
-      velocity="0.5" />
+  <joint name="joint_hand_left" type="prismatic">
+    <origin xyz="0 0 0.0122" rpy="1.5708 0 3.1416" />
+    <parent link="housing_link" />
+    <child link="hand_left_link" />
+    <axis xyz="1 0 0" />
+    <limit lower="0" upper="0.03" effort="120" velocity="0.5" />
   </joint>
-  <link
-    name="finger_left_link">
+  <link name="finger_left_link">
     <inertial>
-      <origin
-        xyz="0.01141 1.453E-08 0.024079"
-        rpy="0 0 0" />
-      <mass
-        value="0.011888" />
-      <inertia
-        ixx="2.4136E-06"
-        ixy="-7.1143E-13"
-        ixz="1.1892E-07"
-        iyy="2.2441E-06"
-        iyz="1.2315E-12"
-        izz="6.7629E-07" />
+      <origin xyz="0.01141 1.453E-08 0.024079" rpy="0 0 0" />
+      <mass value="0.011888" />
+      <inertia ixx="2.4136E-06" ixy="-7.1143E-13" ixz="1.1892E-07" iyy="2.2441E-06" iyz="1.2315E-12" izz="6.7629E-07" />
     </inertial>
     <visual>
-      <origin
-        xyz="0 0 0"
-        rpy="0 0 0" />
+      <origin xyz="0 0 0" rpy="0 0 0" />
       <geometry>
-        <mesh
-          filename="file://$(find melfa_assista_hardware)/meshes/finger_left_link.stl" />
+        <mesh filename="file://$(find melfa_assista_hardware)/meshes/finger_left_link.stl" />
       </geometry>
-      <material
-        name="">
-        <color
-          rgba="0.79216 0.81961 0.93333 1" />
+      <material name="">
+        <color rgba="0.79216 0.81961 0.93333 1" />
       </material>
     </visual>
     <collision>
-      <origin
-        xyz="0 0 0"
-        rpy="0 0 0" />
+      <origin xyz="0 0 0" rpy="0 0 0" />
       <geometry>
-        <mesh
-          filename="file://$(find melfa_assista_hardware)/meshes/finger_left_link.stl" />
+        <mesh filename="file://$(find melfa_assista_hardware)/meshes/finger_left_link.stl" />
       </geometry>
     </collision>
   </link>
-  <joint
-    name="finger_left_joint"
-    type="fixed">
-    <origin
-      xyz="0.0056005 -0.012 0"
-      rpy="-1.5708 0 0" />
-    <parent
-      link="hand_left_link" />
-    <child
-      link="finger_left_link" />
-    <axis
-      xyz="0 0 0" />
+  <joint name="finger_left_joint" type="fixed">
+    <origin xyz="0.0056005 -0.012 0" rpy="-1.5708 0 0" />
+    <parent link="hand_left_link" />
+    <child link="finger_left_link" />
+    <axis xyz="0 0 0" />
   </joint>
-  <link
-    name="hand_right_link">
+  <link name="hand_right_link">
     <inertial>
-      <origin
-        xyz="-0.0011169 -0.015033 0.0033678"
-        rpy="0 0 0" />
-      <mass
-        value="0.0034696" />
-      <inertia
-        ixx="2.1052E-07"
-        ixy="-1.1835E-07"
-        ixz="4.2799E-08"
-        iyy="4.0216E-07"
-        iyz="4.2388E-08"
-        izz="5.2415E-07" />
+      <origin xyz="-0.0011169 -0.015033 0.0033678" rpy="0 0 0" />
+      <mass value="0.0034696" />
+      <inertia ixx="2.1052E-07" ixy="-1.1835E-07" ixz="4.2799E-08" iyy="4.0216E-07" iyz="4.2388E-08" izz="5.2415E-07" />
     </inertial>
     <visual>
-      <origin
-        xyz="0 0 0"
-        rpy="0 0 0" />
+      <origin xyz="0 0 0" rpy="0 0 0" />
       <geometry>
-        <mesh
-          filename="file://$(find melfa_assista_hardware)/meshes/hand_right_link.stl" />
+        <mesh filename="file://$(find melfa_assista_hardware)/meshes/hand_right_link.stl" />
       </geometry>
-      <material
-        name="">
-        <color
-          rgba="0.79216 0.81961 0.93333 1" />
+      <material name="">
+        <color rgba="0.79216 0.81961 0.93333 1" />
       </material>
     </visual>
     <collision>
-      <origin
-        xyz="0 0 0"
-        rpy="0 0 0" />
+      <origin xyz="0 0 0" rpy="0 0 0" />
       <geometry>
-        <mesh
-          filename="file://$(find melfa_assista_hardware)/meshes/hand_right_link.stl" />
+        <mesh filename="file://$(find melfa_assista_hardware)/meshes/hand_right_link.stl" />
       </geometry>
     </collision>
   </link>
-  <joint
-    name="joint_hand_right"
-    type="prismatic">
-    <origin
-      xyz="0 0 0.0122"
-      rpy="1.5708 0 0" />
-    <parent
-      link="housing_link" />
-    <child
-      link="hand_right_link" />
-    <axis
-      xyz="1 0 0" />
-    <limit
-      lower="0"
-      upper="0.03"
-      effort="120"
-      velocity="0.5" />
-    <mimic
-      joint="joint_hand_left"
-      multiplier="1"
-      offset="0" />
+  <joint name="joint_hand_right" type="prismatic">
+    <origin xyz="0 0 0.0122" rpy="1.5708 0 0" />
+    <parent link="housing_link" />
+    <child link="hand_right_link" />
+    <axis xyz="1 0 0" />
+    <limit lower="0" upper="0.03" effort="120" velocity="0.5" />
+    <mimic joint="joint_hand_left" multiplier="1" offset="0" />
   </joint>
-  <link
-    name="finger_right_joint">
+  <link name="finger_right_joint">
     <inertial>
-      <origin
-        xyz="0.01141 1.453E-08 0.024079"
-        rpy="0 0 0" />
-      <mass
-        value="0.013672" />
-      <inertia
-        ixx="2.7756E-06"
-        ixy="-8.1815E-13"
-        ixz="1.3676E-07"
-        iyy="2.5808E-06"
-        iyz="1.4163E-12"
-        izz="7.7774E-07" />
+      <origin xyz="0.01141 1.453E-08 0.024079" rpy="0 0 0" />
+      <mass value="0.013672" />
+      <inertia ixx="2.7756E-06" ixy="-8.1815E-13" ixz="1.3676E-07" iyy="2.5808E-06" iyz="1.4163E-12" izz="7.7774E-07" />
     </inertial>
     <visual>
-      <origin
-        xyz="0 0 0"
-        rpy="0 0 0" />
+      <origin xyz="0 0 0" rpy="0 0 0" />
       <geometry>
-        <mesh
-          filename="file://$(find melfa_assista_hardware)/meshes/finger_right_joint.stl" />
+        <mesh filename="file://$(find melfa_assista_hardware)/meshes/finger_right_joint.stl" />
       </geometry>
-      <material
-        name="">
-        <color
-          rgba="0.79608 0.82353 0.93725 1" />
+      <material name="">
+        <color rgba="0.79608 0.82353 0.93725 1" />
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